File: drivers1.kicad_sch (KiCad schematic)
At the start: 0 parts

Commit message: Play around with drivers
Parts:
- added C1, C2, C3, C4: 470pF, APRLPrints:C_0402, symbol Device:C_Small
- added C10: 100nF, APRLPrints:C_0402, symbol Device:C_Small
- added C5, C6: 68uF, Capacitor_SMD:CP_Elec_10x10.5, symbol Device:C_Small
- added C7, C8: 22nF, APRLPrints:C_0402, symbol Device:C_Small
- added C9: 2.2uF, APRLPrints:C_0603, symbol Device:C_Small
- added J1: Conn_01x04, Connector_JST:JST_XH_B4B-XH-AM_1x04_P2.50mm_Vertical, symbol Connector_Generic:Conn_01x04
- added R1: 24k, APRLPrints:R_0402, symbol Device:R_Small_US
- added U6: TMC2241ATC, libserie:QFN-38_EP_5.63x7.6_Pitch0.5mm, symbol libserie:TMC2241ATC
Connections:
- new net: R1.1, U6.3 (IREF)
- new net: C4.1, J1.1 (Pin_1), U6.24 (OUT2B)
- new net: C8.2, U6.18 (VCP)
- new net: C2.1, J1.3 (Pin_3), U6.27 (OUT2A)
- new net: C1.1, J1.4 (Pin_4), U6.29 (OUT1A)
- new net: C3.1, J1.2 (Pin_2), U6.22 (OUT1B)
- new net: C9.2, U6.5 (VDD18)
- new net: C7.1, U6.17 (CPO)
- new net: C7.2, U6.16 (CPI)
- new net: U6.19 (NC), U6.20 (NC), U6.31 (NC), U6.32 (NC)
- new net +3.3V: C10.2, U6.7 (VCCIO)
- new net DIAG0: U6.14 (DIAG1/SW)
- new net DIAG1: U6.13 (DIAG0)
- new net DIR: U6.2 (DIR)
- new net EP: C1.2, C10.1, C2.2, C3.2, C4.2, C5.2, C6.2, C9.1, R1.2, U6.23 (PGND), U6.28 (PGND), U6.39 (EP), U6.6 (AGND)
- new net MISO: U6.37 (SDO/NAO)
- new net MOSI: U6.36 (SDI/AD0)
- new net SCK: U6.35 (SCK/AD1)
- new net STEP: U6.1 (STEP)
- new net VM: C5.1, C6.1, C8.1, U6.21 (VS), U6.25 (VS), U6.26 (VS), U6.30 (VS)
- new net ~{CS}: U6.34 (~{CS}/AD2)
- new net ~{DRV_EN}: U6.11 (~{DRV_EN})
- new net ~{SLEEP}: U6.33 (~{SLEEP})
- no-connect marks 0 -> 6
Other:
- note added: "+VM Should be polymer caps All caps should be rated for 100V"
- note added: "May be changed to increase current resolution"

Commit message: I dont know whats going on here
Parts:
- added C25: 100nF, Capacitor_SMD:CP_Elec_10x10.5, symbol Device:C_Small
- C6: renamed from C5; value 68uF -> 100uF
- C8: renamed from C6; value 68uF -> 100uF
- renumbered C10 to C1, C4 to C10, C9 to C2, C7 to C3, C8 to C4, C1 to C5, C2 to C7, C3 to C9, U6 to U2
Connections:
- net DIAG0: now also U2.13 (DIAG0); no longer U2.14 (DIAG1/SW)
- net DIAG1: now also U2.14 (DIAG1/SW); no longer U2.13 (DIAG0)
- net EP: now also U2.38 (CLK), C25.2
- net VM: now also C25.1
- net MISO renamed DRV_MISO
- net MOSI renamed DRV_MOSI
- net SCK renamed DRV_SCK
- net ~{SLEEP} renamed ~{DRV_SLEEP}
Other:
- note added: "1%, May be changed to increase current resolution"
- note added: "All caps should be rated for 100V"
- note added: "Driver supports an external clock which affects: 1. Current chopping frequency 2. SPI frequency It may be advisable to expose MCO on the STM32 and drive this pin with it."
- note removed: "+VM Should be polymer caps All caps should be rated for 100V"
- note removed: "May be changed to increase current resolution"
- moved on the sheet: C1, C10, C2, C3, C4, C5, C6, C7, C8, C9, J1, R1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
