File: drivers1.kicad_sch (KiCad schematic)
At the start: 15 parts, among them J31 Conn_01x04, U17 TMC2241ATC

Commit message: ???
Parts:
- renumbered C73 to C78, C74 to C79, C75 to C80, C76 to C81, C77 to C82, C78 to C83, C79 to C84, C80 to C85, C81 to C86, C82 to C87, C83 to C88, C84 to C89, J31 to J29, R51 to R64, U17 to U24
Connections:
- net at C89.1, J29.2 (Pin_2): now also U24.22 (OUT1B); no longer U24.24 (OUT2B)
- net at C87.1, J29.1 (Pin_1): now also U24.24 (OUT2B); no longer U24.22 (OUT1B)

Commit message: loadcell math coming soon(tm)
Parts:
- removed C88: 100uF, Capacitor_SMD:CP_Elec_10x10.5, symbol Device:C_Small
- renumbered C80 to C78, C81 to C79, C82 to C80, C84 to C81, C86 to C82, C85 to C84, C87 to C85, C89 to C86, C78 to C87, C79 to C88, J29 to J28, R64 to R76, U24 to U22
Connections:
- net ~{DRV_EN} is gone; now on net EP: U22.11 (DRV_EN)
- net ~{DRV_SLEEP} is gone; now on net +3.3V: U22.33 (~{SLEEP})
- now unconnected: U22.19 (NC), U22.20 (NC), U22.31 (NC), U22.32 (NC)
Other:
- moved on the sheet: C80, C81, C82

Commit message: a
Parts:
- added C84: 100nF, APRLPrints:C_0603, symbol Device:C_Small
- J24: renamed from J28; footprint Connector_JST:JST_XH_B4B-XH-AM_1x04_P2.50mm_Vertical -> libserie:JST_XH_B4B-XH-AM_1x04_P2.50mm_Vertical
- renumbered C78 to C82, C79 to C83, C80 to C85, C81 to C86, C82 to C87, C83 to C88, C84 to C89, C85 to C90, C86 to C91, C87 to C92, C88 to C93, R76 to R75, U22 to U24
Connections:
- net EP: now also C84.2
- net VM: now also C84.1
- net at C91.1, U24.22 (OUT1B): now also J24.1 (Pin_1); no longer J24.2 (Pin_2)
- net at C89.1, U24.29 (OUT1A): now also J24.4 (Pin_4); no longer J24.3 (Pin_3)
- net at C88.1, U24.27 (OUT2A): now also J24.3 (Pin_3); no longer J24.4 (Pin_4)
- net at C90.1, U24.24 (OUT2B): now also J24.2 (Pin_2); no longer J24.1 (Pin_1)
- net DIAG1: no longer names the net of U24.14 (DIAG1/SW)
- no-connect marks 6 -> 7
Other:
- note added: "Only 1 diag pin is used"
- moved on the sheet: C85, C86, C87
