File: poweroutputs.kicad_sch (KiCad schematic)
At the start: 53 parts, among them J12 Screw_Terminal_01x02, J2 Screw_Terminal_01x02, J3 Screw_Terminal_01x02, J4 Screw_Terminal_01x02, J5 Screw_Terminal_01x02, J6 Screw_Terminal_01x02, J7 Screw_Terminal_01x02, Q1 AO3400A, Q2 Si7450DP, Q3 Si7450DP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

Commit message: Soften scope, begin layout, reorganize sheets (still need to delete extras)
Parts:
- removed D11, D14, D16: SS54, Diode_SMD:D_SMA, symbol Diode:SS38
- removed D12, D13, D15: LED_Small, symbol Device:LED_Small
- removed J12, J6, J7: Screw_Terminal_01x02, symbol Connector:Screw_Terminal_01x02
- removed Q1, Q6, Q7: AO3400A, Package_TO_SOT_SMD:SOT-23, symbol Transistor_FET:AO3400A
- removed R30, R40, R43: 100k, symbol Device:R_Small_US
- removed R33, R35, R42: 10k, symbol Device:R_Small_US
- removed R34, R41, R6: 10R, symbol Device:R_Small_US
Other:
- note removed: "Low Power Outputs"
