File: Serie.kicad_sch (KiCad schematic)
At the start: 0 parts

Commit message: I dont know whats going on here
Other:
- removed sheet Board IO
- removed sheet Driver Set 1
- removed sheet Driver Set 2
- removed sheet Power
- removed sheet Thermocouples
- added sheet Changelog and Notes (chagenotes.kicad_sch)
- added sheet Connections (connections.kicad_sch)
- note added: "Serie 3D Printer Mainboard"
Changed lines of the file:
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@@
 		(company "Nolan and Kanin")
 	)
+	(text "Serie 3D Printer Mainboard"
+		(exclude_from_sim no)
+		(at 137.414 28.956 0)
+		(effects
+			(font
+				(size 6.35 6.35)
+				(thickness 1.27)
+				(bold yes)
+			)
+		)
+	)
 	(sheet
-		(at 88.9 137.16)
-		(size 53.34 27.94)
+		(at 100.33 135.89)
+		(size 35.56 20.32)
 		(exclude_from_sim no)
 		(in_bom yes)
@@
 			(color 0 0 0 0.0000)
 		)
-		(property "Sheetname" "Thermocouples"
-			(at 88.9 136.4484 0)
+		(property "Sheetname" "Connections"
+			(at 100.33 135.1784 0)
 			(effects
 				(font
@@
 			)
 		)
-		(property "Sheetfile" "thermocouples.kicad_sch"
-			(at 88.9 165.6846 0)
-			(effects
-				(font
-					(size 1.27 1.27)
-				)
-				(justify left top)
-			)
-		)
-		(instances
-			(project "Serie"
-				(path "/8fdbc9dc-a02a-488d-a5a6-6a3827681e3b"
-					(page "5")
-				)
-			)
-		)
-	)
-	(sheet
-		(at 146.05 95.25)
-		(size 66.04 33.02)
-		(exclude_from_sim no)
-		(in_bom yes)
-		(on_board yes)
-		(dnp no)
-		(fields_autoplaced yes)
-		(stroke
-			(width 0.1524)
-			(type solid)
-		)
-		(fill
-			(color 0 0 0 0.0000)
-		)
-		(property "Sheetname" "Power"
-			(at 146.05 94.5384 0)
-			(effects
-				(font
-					(size 1.27 1.27)
-				)
-				(justify left bottom)
-			)
-		)
-		(property "Sheetfile" "power.kicad_sch"
-			(at 146.05 128.8546 0)
+		(property "Sheetfile" "connections.kicad_sch"
+			(at 100.33 156.7946 0)
 			(effects
 				(font
@@
 	)
 	(sheet
-		(at 214.63 95.25)
-		(size 46.99 30.48)
+		(at 140.97 135.89)
+		(size 34.29 20.32)
 		(exclude_from_sim no)
 		(in_bom yes)
@@
 			(color 0 0 0 0.0000)
 		)
-		(property "Sheetname" "Board IO"
-			(at 214.63 94.5384 0)
+		(property "Sheetname" "Changelog and Notes"
+			(at 140.97 135.1784 0)
 			(effects
 				(font
@@
 			)
 		)
-		(property "Sheetfile" "io.kicad_sch"
-			(at 214.63 126.3146 0)
-			(effects
-				(font
-					(size 1.27 1.27)
-				)
-				(justify left top)
-			)
-		)
-		(instances
-			(project "Serie"
-				(path "/8fdbc9dc-a02a-488d-a5a6-6a3827681e3b"
-					(page "6")
-				)
-			)
-		)
-	)
-	(sheet
-		(at 146.05 133.35)
-		(size 66.04 29.21)
-		(exclude_from_sim no)
-		(in_bom yes)
-		(on_board yes)
-		(dnp no)
-		(fields_autoplaced yes)
-		(stroke
-			(width 0.1524)
-			(type solid)
-		)
-		(fill
-			(color 0 0 0 0.0000)
-		)
-		(property "Sheetname" "Driver Set 1"
-			(at 146.05 132.6384 0)
-			(effects
-				(font
-					(size 1.27 1.27)
-				)
-				(justify left bottom)
-			)
-		)
-		(property "Sheetfile" "drivers1.kicad_sch"
-			(at 146.05 163.1446 0)
+		(property "Sheetfile" "chagenotes.kicad_sch"
+			(at 140.97 156.7946 0)
 			(effects
 				(font
@@
 				)
 			)
-		)
-	)
-	(sheet
-		(at 215.9 134.62)
-		(size 46.99 29.21)
-		(exclude_from_sim no)
-		(in_bom yes)
-		(on_board yes)
-		(dnp no)
-		(fields_autoplaced yes)
-		(stroke
-			(width 0.1524)
-			(type solid)
-		)
-		(fill
-			(color 0 0 0 0.0000)
-		)
-		(property "Sheetname" "Driver Set 2"
-			(at 215.9 133.9084 0)
-			(effects
-				(font
-					(size 1.27 1.27)
-				)
-				(justify left bottom)
-			)
-		)
-		(property "Sheetfile" "drivers2.kicad_sch"
-			(at 215.9 164.4146 0)
-			(effects
-				(font
-					(size 1.27 1.27)
-				)
-				(justify left top)
-			)
-		)
-		(instances
-			(project "Serie"
-				(path "/8fdbc9dc-a02a-488d-a5a6-6a3827681e3b"
-					(page "4")
-				)
-			)

Commit message: ???
Parts:
- added H1, H2, H3, H4: MountingHole, MountingHole:MountingHole_3.2mm_M3, symbol Mechanical:MountingHole
Other:
- note added: "Mounting Holes"
