File: chagenotes.kicad_sch (KiCad schematic)
At the start: 0 parts

Commit message: loadcell math coming soon(tm)
Other:
- note removed: "There are only 7 unique sheets, most of which is stuff I pinched from past projects or is already extremely simple"
Changed lines of the file:
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@@
 		(company "Nolan and Kanin")
 	)
-	(text "There are only 7 unique sheets, most of which is stuff I pinched from past projects or is already extremely simple"
-		(exclude_from_sim no)
-		(at 123.19 69.85 0)
-		(effects
-			(font
-				(size 1.27 1.27)
-			)
-		)
-	)
 )
