File: Serie.kicad_pcb (KiCad board)
At the start: 2 copper layers, 18 parts, among them J1 Conn_01x04, U1 STM32H723ZGTx, U2 MAX31865xTP, U3 MAX31865xTP, U4 MAX31865xTP, U5 MAX31865xTP, U6 TMC2241ATC

Commit message: Soften scope, begin layout, reorganize sheets (still need to delete extras)
Parts:
- added C100: 22nF, APRLPrints:C_0603, F.Cu at (140.0, 38.2)
- added C101: 100nF, APRLPrints:C_0603, F.Cu at (131.9, 36.1)
- added C102: 470pF, APRLPrints:C_0603, F.Cu at (130.6, 29.2)
- added C103: 100nF, APRLPrints:C_0603, F.Cu at (137.4, 36.2)
- added C104: 470pF, APRLPrints:C_0603, F.Cu at (133.4, 29.2)
- added C105: 100uF, Capacitor_SMD:CP_Elec_10x10.5, F.Cu at (124.4, 35.4)
- added C106: 470pF, APRLPrints:C_0603, F.Cu at (138.7, 29.2)
- added C107: 100uF, Capacitor_SMD:CP_Elec_10x10.5, F.Cu at (124.4, 46.5)
- added C108: 470pF, APRLPrints:C_0603, F.Cu at (136.1, 29.2)
- added C109: 100nF, APRLPrints:C_0603, F.Cu at (157.9, 45.9)
- added C11: 100nF, APRLPrints:C_0603, F.Cu at (200.8, 69.4)
- added C110: 2.2uF, APRLPrints:C_0603, F.Cu at (156.4, 45.9)
- added C111: 22nF, APRLPrints:C_0603, F.Cu at (162.0, 40.9)
- added C112: 22nF, APRLPrints:C_0603, F.Cu at (162.0, 38.2)
- added C113: 100nF, APRLPrints:C_0603, F.Cu at (159.4, 36.0)
- added C114: 470pF, APRLPrints:C_0603, F.Cu at (152.6, 29.0)
- added C115: 100nF, APRLPrints:C_0603, F.Cu at (153.9, 35.9)
- added C116: 470pF, APRLPrints:C_0603, F.Cu at (155.4, 29.0)
- added C117: 100uF, Capacitor_SMD:CP_Elec_10x10.5, F.Cu at (146.4, 35.2)
- added C118: 470pF, APRLPrints:C_0603, F.Cu at (160.7, 29.0)
- added C119: 100uF, Capacitor_SMD:CP_Elec_10x10.5, F.Cu at (146.4, 46.3)
- added C12: 10pF, APRLPrints:C_0603, F.Cu at (182.1, 72.0)
- added C120: 470pF, APRLPrints:C_0603, F.Cu at (158.1, 29.0)
- added C121: 100nF, APRLPrints:C_0603, F.Cu at (91.8, 46.0)
- added C122: 2.2uF, APRLPrints:C_0603, F.Cu at (90.3, 46.0)
- added C123: 22nF, APRLPrints:C_0603, F.Cu at (95.8, 41.0)
- added C124: 22nF, APRLPrints:C_0603, F.Cu at (95.8, 38.4)
- added C125: 100nF, APRLPrints:C_0603, F.Cu at (93.2, 36.1)
- added C126: 470pF, APRLPrints:C_0603, F.Cu at (86.4, 29.1)
- added C127: 100nF, APRLPrints:C_0603, F.Cu at (87.7, 36.0)
- added C128: 470pF, APRLPrints:C_0603, F.Cu at (89.2, 29.1)
- added C129: 100uF, Capacitor_SMD:CP_Elec_10x10.5, F.Cu at (80.2, 46.4)
- added C13: 22uF, APRLPrints:C_0805, F.Cu at (205.4, 79.5)
- added C130: 470pF, APRLPrints:C_0603, F.Cu at (94.5, 29.1)
- added C131: 100uF, Capacitor_SMD:CP_Elec_10x10.5, F.Cu at (80.2, 35.3)
- added C132: 470pF, APRLPrints:C_0603, F.Cu at (91.9, 29.1)
- added C133: 100nF, APRLPrints:C_0603, F.Cu at (114.0, 46.0)
- added C134: 2.2uF, APRLPrints:C_0603, F.Cu at (112.5, 46.0)
- added C135: 22nF, APRLPrints:C_0603, F.Cu at (118.0, 41.0)
- added C136: 22nF, APRLPrints:C_0603, F.Cu at (118.0, 38.4)
- added C137: 100nF, APRLPrints:C_0603, F.Cu at (109.9, 36.1)
- added C138: 470pF, APRLPrints:C_0603, F.Cu at (108.6, 29.2)
- added C139: 100nF, APRLPrints:C_0603, F.Cu at (115.4, 36.2)
- added C14: 10pF, APRLPrints:C_0603, F.Cu at (182.1, 74.6)
- added C140: 470pF, APRLPrints:C_0603, F.Cu at (111.4, 29.2)
- added C141: 100uF, Capacitor_SMD:CP_Elec_10x10.5, F.Cu at (102.4, 46.5)
- added C142: 470pF, APRLPrints:C_0603, F.Cu at (116.7, 29.2)
- added C143: 100uF, Capacitor_SMD:CP_Elec_10x10.5, F.Cu at (102.4, 35.4)
- added C144: 470pF, APRLPrints:C_0603, F.Cu at (114.1, 29.2)
- added C145: 100nF, APRLPrints:C_0603, F.Cu at (-4.63, 106.0)
- added C146: 100nF, APRLPrints:C_0603, F.Cu at (-4.65, 133.0)
- added C15: 22uF, APRLPrints:C_0805, F.Cu at (198.6, 79.4)
- added C16: 100nF, APRLPrints:C_0603, F.Cu at (184.1, 69.2)
- added C17: 100nF, APRLPrints:C_0603, F.Cu at (193.4, 79.0)
- added C18: 100nF, APRLPrints:C_0603, F.Cu at (196.3, 69.8)
- added C19: 100nF, APRLPrints:C_0603, F.Cu at (187.0, 66.7)
- added C20: 100nF, APRLPrints:C_0603, F.Cu at (184.1, 74.8)
- added C21: 100nF, APRLPrints:C_0603, F.Cu at (111.2, 76.0)
- added C22: 22uF, APRLPrints:C_0805, F.Cu at (86.4, 80.0)
- added C23: 100nF, APRLPrints:C_0603, F.Cu at (110.6, 84.6)
- added C24: 22uF, APRLPrints:C_0805, F.Cu at (86.4, 82.0)
- added C25: 22uF, APRLPrints:C_0805, F.Cu at (86.4, 84.0)
- added C26: 100nF, APRLPrints:C_0603, F.Cu at (114.1, 65.2)
- added C28: 22uF, APRLPrints:C_0805, F.Cu at (94.3, 87.1)
- added C29: 100nF, APRLPrints:C_0603, F.Cu at (121.6, 64.4)
- added C30: 100nF, APRLPrints:C_0603, F.Cu at (137.2, 75.4)
- added C31: 22uF, APRLPrints:C_0805, F.Cu at (96.2, 87.1)
- added C32: 100nF, APRLPrints:C_0603, F.Cu at (127.6, 90.8)
- added C33: 100nF, APRLPrints:C_0603, F.Cu at (137.0, 81.4)
- added C34: 22uF, APRLPrints:C_0805, F.Cu at (98.1, 87.1)
- added C35: 100nF, APRLPrints:C_0603, F.Cu at (133.6, 90.2)
- added C36: 100nF, APRLPrints:C_0603, F.Cu at (126.6, 64.6)
- added C37: 100nF, APRLPrints:C_0603, F.Cu at (90.1, 90.9)
- added C38: 100nF, APRLPrints:C_0603, F.Cu at (136.4, 68.3)
- added C39: 100nF, APRLPrints:C_0603, F.Cu at (122.4, 90.6)
- added C40: 100nF, APRLPrints:C_0603, F.Cu at (116.0, 90.8)
- added C41: 22uF, APRLPrints:C_0805, F.Cu at (104.5, 87.1)
- added C42: 22uF, APRLPrints:C_0805, F.Cu at (90.5, 80.0)
- added C43: 22uF, APRLPrints:C_0805, F.Cu at (106.5, 87.1)
- added C44: 22uF, APRLPrints:C_0805, F.Cu at (90.5, 82.0)
- added C45: 22uF, APRLPrints:C_0805, F.Cu at (108.5, 87.1)
- added C46: 22uF, APRLPrints:C_0805, F.Cu at (90.5, 84.0)
- added C47: 2.2uF, APRLPrints:C_0603, F.Cu at (132.8, 91.8)
- added C48: 2.2uF, APRLPrints:C_0603, F.Cu at (138.0, 69.0)
- added C49: 100nF, APRLPrints:C_0603, F.Cu at (110.8, 86.2)
- added C51: 10pF, APRLPrints:C_0603, F.Cu at (101.0, 78.4)
- added C52: 10pF, APRLPrints:C_0603, F.Cu at (101.2, 83.5)
- added C53: 10n, APRLPrints:C_0603, F.Cu at (207.0, 107.6)
- added C54: 100n, APRLPrints:C_0603, F.Cu at (207.0, 110.4)
- added C55: 10n, APRLPrints:C_0603, F.Cu at (207.0, 113.2)
- added C56: 100n, APRLPrints:C_0603, F.Cu at (204.1, 106.4)
- added C57: 100n, APRLPrints:C_0603, F.Cu at (197.2, 106.8)
- added C58: 10n, APRLPrints:C_0603, F.Cu at (207.0, 140.5)
- added C59: 100n, APRLPrints:C_0603, F.Cu at (207.0, 143.3)
- added C60: 10n, APRLPrints:C_0603, F.Cu at (207.0, 146.1)
- added C61: 100n, APRLPrints:C_0603, F.Cu at (197.2, 139.7)
- added C62: 100n, APRLPrints:C_0603, F.Cu at (204.1, 139.3)
- added C63: 10n, APRLPrints:C_0603, F.Cu at (207.0, 129.6)
- added C64: 100n, APRLPrints:C_0603, F.Cu at (207.0, 132.4)
- added C65: 10n, APRLPrints:C_0603, F.Cu at (207.0, 135.2)
- added C66: 100n, APRLPrints:C_0603, F.Cu at (197.2, 128.8)
- added C67: 100n, APRLPrints:C_0603, F.Cu at (204.1, 128.4)
- added C68: 10n, APRLPrints:C_0603, F.Cu at (207.0, 118.5)
- added C69: 100n, APRLPrints:C_0603, F.Cu at (207.0, 121.3)
- added C70: 10n, APRLPrints:C_0603, F.Cu at (207.0, 124.1)
- added C71: 100n, APRLPrints:C_0603, F.Cu at (204.1, 117.3)
- added C72: 100n, APRLPrints:C_0603, F.Cu at (197.2, 117.7)
- added C73: 100nF, APRLPrints:C_0603, F.Cu at (201.7, 46.0)
- added C74: 2.2uF, APRLPrints:C_0603, F.Cu at (200.2, 46.0)
- added C75: 22nF, APRLPrints:C_0603, F.Cu at (205.7, 40.7)
- added C76: 22nF, APRLPrints:C_0603, F.Cu at (205.7, 38.0)
- added C77: 100nF, APRLPrints:C_0603, F.Cu at (203.1, 36.2)
- added C78: 470pF, APRLPrints:C_0603, F.Cu at (196.3, 29.2)
- added C79: 100nF, APRLPrints:C_0603, F.Cu at (197.6, 36.1)
- added C80: 470pF, APRLPrints:C_0603, F.Cu at (199.1, 29.2)
- added C81: 100uF, Capacitor_SMD:CP_Elec_10x10.5, F.Cu at (190.1, 46.5)
- added C82: 470pF, APRLPrints:C_0603, F.Cu at (204.4, 29.2)
- added C83: 100uF, Capacitor_SMD:CP_Elec_10x10.5, F.Cu at (190.1, 35.4)
- added C84: 470pF, APRLPrints:C_0603, F.Cu at (201.8, 29.2)
- added C85: 100nF, APRLPrints:C_0603, F.Cu at (179.8, 46.0)
- added C86: 2.2uF, APRLPrints:C_0603, F.Cu at (178.3, 46.0)
- added C87: 22nF, APRLPrints:C_0603, F.Cu at (183.9, 40.9)
- added C88: 22nF, APRLPrints:C_0603, F.Cu at (183.9, 38.2)
- added C89: 100nF, APRLPrints:C_0603, F.Cu at (181.3, 36.2)
- added C90: 470pF, APRLPrints:C_0603, F.Cu at (174.5, 29.2)
- added C91: 100nF, APRLPrints:C_0603, F.Cu at (175.8, 36.1)
- added C92: 470pF, APRLPrints:C_0603, F.Cu at (177.3, 29.2)
- added C93: 100uF, Capacitor_SMD:CP_Elec_10x10.5, F.Cu at (168.3, 46.5)
- added C94: 470pF, APRLPrints:C_0603, F.Cu at (182.6, 29.2)
- added C95: 100uF, Capacitor_SMD:CP_Elec_10x10.5, F.Cu at (168.3, 35.4)
- added C96: 470pF, APRLPrints:C_0603, F.Cu at (180.0, 29.2)
- added C97: 100nF, APRLPrints:C_0603, F.Cu at (135.9, 46.0)
- added C98: 2.2uF, APRLPrints:C_0603, F.Cu at (134.4, 46.0)
- added C99: 22nF, APRLPrints:C_0603, F.Cu at (140.0, 40.9)
- added D1: LED_Small, APRLPrints:LED_0603, F.Cu at (212.5, 53.5)
- added D10: LED_Small, APRLPrints:LED_0603, F.Cu at (107.8, 84.2)
- added D11: SS54, Diode_SMD:D_SMA, F.Cu at (94.5, 81.4)
- added D13: SS54, Diode_SMD:D_SMA, F.Cu at (-23.0, 148.7)
- added D14: LED_Small, APRLPrints:LED_0603, F.Cu at (22.4, 227.3)
- added D15: SS54, Diode_SMD:D_SMA, F.Cu at (20.4, 232.3)
- added D16: LED, APRLPrints:LED_0603, F.Cu at (197.0, 112.2)
- added D17: LED, APRLPrints:LED_0603, F.Cu at (197.0, 145.1)
- added D18: LED, APRLPrints:LED_0603, F.Cu at (197.0, 134.2)
- added D19: LED, APRLPrints:LED_0603, F.Cu at (197.0, 123.1)
- added D2: PMEG3010BER, Diode_SMD:Nexperia_CFP3_SOD-123W, F.Cu at (204.5, 53.5)
- added D20: LED_Small, APRLPrints:LED_0603, F.Cu at (-9.25, 107.3)
- added D21: LED_Small, APRLPrints:LED_0603, F.Cu at (-9.23, 94.1)
- added D22: SS54, Diode_SMD:D_SMA, F.Cu at (-7.63, 110.3)
- added D23: SS54, Diode_SMD:D_SMA, F.Cu at (-7.63, 96.9)
- added D24: LED_Small, APRLPrints:LED_0603, F.Cu at (-9.27, 134.4)
- added D25: LED_Small, APRLPrints:LED_0603, F.Cu at (-9.25, 121.1)
- added D26: SS54, Diode_SMD:D_SMA, F.Cu at (-7.65, 137.4)
- added D27: SS54, Diode_SMD:D_SMA, F.Cu at (-7.65, 123.9)
- added D28: LED_Small, APRLPrints:LED_0603, F.Cu at (4.95, 216.3)
- added D29: SS54, Diode_SMD:D_SMA, F.Cu at (2.92, 221.3)
- added D3: LED_Small, APRLPrints:LED_0603, F.Cu at (213.9, 79.6)
- added D30: LED_Small, APRLPrints:LED_0603, F.Cu at (39.6, 227.4)
- added D31: SS54, Diode_SMD:D_SMA, F.Cu at (37.5, 232.4)
- added D32: LED_Small, APRLPrints:LED_0603, F.Cu at (39.5, 216.2)
- added D33: SS54, Diode_SMD:D_SMA, F.Cu at (37.5, 221.2)
- added D34: LED_Small, APRLPrints:LED_0603, F.Cu at (4.95, 227.3)
- added D35: SS54, Diode_SMD:D_SMA, F.Cu at (2.92, 232.3)
- added D36: LED_Small, APRLPrints:LED_0603, F.Cu at (22.5, 216.5)
- added D37: SS54, Diode_SMD:D_SMA, F.Cu at (20.5, 221.5)
- added D4: PMEG3010BER, Diode_SMD:Nexperia_CFP3_SOD-123W, F.Cu at (207.8, 80.2)
- added D5: LED_Small, APRLPrints:LED_0603, F.Cu at (190.9, 66.0)
- added D6: LED_Small, APRLPrints:LED_0603, F.Cu at (204.0, 82.5)
- added D7: LED_Small, APRLPrints:LED_0603, F.Cu at (198.1, 74.8)
- added D8: SS54, Diode_SMD:D_SMA, F.Cu at (71.2, 55.5)
- added D9: SS54, Diode_SMD:D_SMA, F.Cu at (71.1, 72.9)
- added F1: 500mA, Fuse:Fuse_0805_2012Metric, F.Cu at (209.5, 54.0)
- added F2: 500mA, Fuse:Fuse_0805_2012Metric, F.Cu at (210.3, 79.6)
- added F3: XF-508P-B-B, Fuse:Fuseholder_Blade_Mini_Keystone_3568, F.Cu at (81.1, 57.2)
- added F4: XFCN XF-508P-B-B, Fuse:Fuseholder_Blade_Mini_Keystone_3568, F.Cu at (81.2, 74.5)
- added F6: XF-508P-B-B, Fuse:Fuseholder_Blade_Mini_Keystone_3568, F.Cu at (-6.93, 150.1)
- added J10: Conn_01x02, Connector_Molex:Molex_Micro-Fit_3.0_43650-0215_1x02_P3.00mm_Vertical, F.Cu at (14.9, 229.8)
- added J11: Conn_01x03, Connector_Molex:Molex_Micro-Fit_3.0_43650-0315_1x03_P3.00mm_Vertical, F.Cu at (110.9, 213.0)
- added J12: Conn_01x03, Connector_Molex:Molex_Micro-Fit_3.0_43650-0315_1x03_P3.00mm_Vertical, F.Cu at (110.9, 206.0)
- added J13: Conn_01x03, Connector_Molex:Molex_Micro-Fit_3.0_43650-0315_1x03_P3.00mm_Vertical, F.Cu at (110.9, 199.0)
- added J14: Conn_01x03, Connector_Molex:Molex_Micro-Fit_3.0_43650-0315_1x03_P3.00mm_Vertical, F.Cu at (110.9, 192.1)
- added J15: Conn_01x03, Connector_Molex:Molex_Micro-Fit_3.0_43650-0315_1x03_P3.00mm_Vertical, F.Cu at (138.9, 213.0)
- added J16: Conn_01x03, Connector_Molex:Molex_Micro-Fit_3.0_43650-0315_1x03_P3.00mm_Vertical, F.Cu at (138.9, 206.0)
- added J17: Conn_01x03, Connector_Molex:Molex_Micro-Fit_3.0_43650-0315_1x03_P3.00mm_Vertical, F.Cu at (138.9, 199.0)
- added J18: Conn_01x03, Connector_Molex:Molex_Micro-Fit_3.0_43650-0315_1x03_P3.00mm_Vertical, F.Cu at (138.9, 192.0)
- added J19: Conn_01x03, Connector_Molex:Molex_Micro-Fit_3.0_43650-0315_1x03_P3.00mm_Vertical, F.Cu at (96.9, 192.1)
- added J2: USB_C_Receptacle_USB2.0_16P, Connector_USB:USB_C_Receptacle_HRO_TYPE-C-31-M-12, F.Cu at (211.0, 60.8)
- added J20: Conn_01x03, Connector_Molex:Molex_Micro-Fit_3.0_43650-0315_1x03_P3.00mm_Vertical, F.Cu at (96.9, 199.0)
- added J21: Conn_01x03, Connector_Molex:Molex_Micro-Fit_3.0_43650-0315_1x03_P3.00mm_Vertical, F.Cu at (96.9, 206.0)
- added J22: Conn_01x03, Connector_Molex:Molex_Micro-Fit_3.0_43650-0315_1x03_P3.00mm_Vertical, F.Cu at (96.9, 213.0)
- added J23: Conn_01x03, Connector_Molex:Molex_Micro-Fit_3.0_43650-0315_1x03_P3.00mm_Vertical, F.Cu at (124.9, 213.0)
- added J24: Conn_01x03, Connector_Molex:Molex_Micro-Fit_3.0_43650-0315_1x03_P3.00mm_Vertical, F.Cu at (124.9, 206.0)
- added J25: Conn_01x03, Connector_Molex:Molex_Micro-Fit_3.0_43650-0315_1x03_P3.00mm_Vertical, F.Cu at (124.9, 199.0)
- added J26: Conn_01x03, Connector_Molex:Molex_Micro-Fit_3.0_43650-0315_1x03_P3.00mm_Vertical, F.Cu at (124.9, 192.0)
- added J27: Conn_01x02, Connector_Molex:Molex_Micro-Fit_3.0_43650-0215_1x02_P3.00mm_Vertical, F.Cu at (211.2, 111.9)
- added J28: Conn_01x02, Connector_Molex:Molex_Micro-Fit_3.0_43650-0215_1x02_P3.00mm_Vertical, F.Cu at (211.2, 144.8)
- added J29: Conn_01x02, Connector_Molex:Molex_Micro-Fit_3.0_43650-0215_1x02_P3.00mm_Vertical, F.Cu at (211.2, 133.9)
- added J3: RJ45_Hanrun_HR911105A_Horizontal, Connector_RJ:RJ45_Hanrun_HR911105A_Horizontal, F.Cu at (197.1, 98.1)
- added J30: Conn_01x02, Connector_Molex:Molex_Micro-Fit_3.0_43650-0215_1x02_P3.00mm_Vertical, F.Cu at (211.2, 122.8)
- added J31: Conn_01x04, Connector_JST:JST_XH_B4B-XH-AM_1x04_P2.50mm_Vertical, F.Cu at (204.2, 25.3)
- added J32: Conn_01x04, Connector_JST:JST_XH_B4B-XH-AM_1x04_P2.50mm_Vertical, F.Cu at (182.3, 25.3)
- added J33: Conn_01x04, Connector_JST:JST_XH_B4B-XH-AM_1x04_P2.50mm_Vertical, F.Cu at (138.4, 25.3)
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Connections:
- net DIAG1 renamed /Connections/Debugger/TGT_RX
- C1 pad 1: Net-(J1-Pin_4) -> +3.3V
- C10 pad 1: GND -> Net-(U3-VBUS)
- C10 pad 2: +3.3V -> GND
- C2 pad 1: Net-(J1-Pin_3) -> Net-(U2-XTAL1/CLKIN)
- C3 pad 1: Net-(J1-Pin_2) -> +3.3V
- C4 pad 1: Net-(J1-Pin_1) -> Net-(U2-XTAL2)
- C5 pad 1: VM -> +3.3V
- C6 pad 1: VM -> +3.3V
- C7 pad 1: Net-(U6-CPO) -> Net-(U2-VDDCR)
- C7 pad 2: Net-(U6-CPI) -> GND
- C8 pad 1: VM -> Net-(U2-VDDCR)
- C8 pad 2: Net-(U6-VCP) -> GND
- C9 pad 1: GND -> +3.3V
- C9 pad 2: Net-(U6-VDD18) -> GND
- J1 pad 1: Net-(J1-Pin_1) -> +3.3V
- J1 pad 2: Net-(J1-Pin_2) -> /Connections/Connectivity/SWDIO
- J1 pad 3: Net-(J1-Pin_3) -> GND
- J1 pad 4: Net-(J1-Pin_4) -> /Connections/Connectivity/SWCLK
- R1 pad 1: Net-(U6-IREF) -> GND
- R1 pad 2: GND -> Net-(U2-RXER/PHYAD0)
- U1 pad 106: unconnected-(U1H-VCAP-Pad106) -> Net-(C48-Pad2)
- U1 pad 107: Net-(U1I-VSS-Pad107) -> GND
- U1 pad 108: unconnected-(U1I-VDD-Pad108) -> +3.3V
- U1 pad 120: Net-(U1I-VSS-Pad107) -> GND
- U1 pad 121: unconnected-(U1I-VDD-Pad121) -> +3.3V
- U1 pad 130: Net-(U1I-VSS-Pad107) -> GND
- U1 pad 131: unconnected-(U1I-VDD-Pad131) -> +3.3V
- U1 pad 138: unconnected-(U1H-BOOT0-Pad138) -> GND
- U1 pad 143: unconnected-(U1H-PDR_ON-Pad143) -> +3.3V
- U1 pad 144: unconnected-(U1I-VDD-Pad144) -> +3.3V
- U1 pad 16: Net-(U1I-VSS-Pad107) -> GND
- U1 pad 17: unconnected-(U1I-VDD-Pad17) -> +3.3V
- U1 pad 23: unconnected-(U1H-PH0-Pad23) -> Net-(U1H-PH0)
- U1 pad 24: unconnected-(U1H-PH1-Pad24) -> Net-(U1H-PH1)
- U1 pad 25: unconnected-(U1H-NRST-Pad25) -> Net-(U1H-NRST)
- U1 pad 30: unconnected-(U1I-VDD-Pad30) -> +3.3V
- U1 pad 31: unconnected-(U1I-VSSA-Pad31) -> GND
- U1 pad 32: unconnected-(U1H-VREF+-Pad32) -> +3.3V
- U1 pad 33: unconnected-(U1I-VDDA-Pad33) -> +3.3V
- U1 pad 38: Net-(U1I-VSS-Pad107) -> GND
- U1 pad 39: unconnected-(U1I-VDD-Pad39) -> +3.3V
- U1 pad 51: Net-(U1I-VSS-Pad107) -> GND
- U1 pad 52: unconnected-(U1I-VDD-Pad52) -> +3.3V
- U1 pad 6: unconnected-(U1I-VBAT-Pad6) -> +3.3V
- U1 pad 61: Net-(U1I-VSS-Pad107) -> GND
- U1 pad 62: unconnected-(U1I-VDD-Pad62) -> +3.3V
- U1 pad 71: unconnected-(U1H-VCAP-Pad71) -> Net-(C47-Pad2)
- U1 pad 72: unconnected-(U1I-VDD-Pad72) -> +3.3V
- U1 pad 83: Net-(U1I-VSS-Pad107) -> GND
- U1 pad 84: unconnected-(U1I-VDD-Pad84) -> +3.3V
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Routing:
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- added copper zone on B.Cu, net /Connections/High Power Outputs 1/High Power Output Set 1/PWR
- added copper zone on F.Cu, net /Connections/High Power Outputs 1/High Power Output Set 1/PWR
- added copper zone on In1.Cu, net /Connections/High Power Outputs 1/High Power Output Set 1/PWR
- added copper zone on In2.Cu, net /Connections/High Power Outputs 1/High Power Output Set 1/PWR
- added copper zone on F.Cu, net GND
- added copper zone on B.Cu, net Net-(D24-K)
- added copper zone on F.Cu, net Net-(D24-K)
- added copper zone on In1.Cu, net Net-(D24-K)
- added copper zone on In2.Cu, net Net-(D24-K)
- added copper zone on B.Cu, net Net-(D25-K)
- added copper zone on F.Cu, net Net-(D25-K)
- added copper zone on In1.Cu, net Net-(D25-K)
- added copper zone on In2.Cu, net Net-(D25-K)
- added copper zone on B.Cu, net Net-(J9-Pin_2)
- added copper zone on F.Cu, net Net-(J9-Pin_2)
- added copper zone on In1.Cu, net Net-(J9-Pin_2)
- added copper zone on In2.Cu, net Net-(J9-Pin_2)
Other:
- board outline added: 159 x 140 mm
- copper layers 2 -> 4

Commit message: ???
Parts:
- removed C1, C7: 1uF, APRLPrints:C_0603
- removed C10, C101, C103, C109, C11, C113, C115, C121, C125, C127, C133, C137, C139, C145, C146, C16, C17, C18, C19, C20, C21, C23, C26, C29, C3, C30, C32, C33, C35, C36, C37, C38, C39, C40, C49, C5, C6, C73, C77, C79, C85, C89, C91, C97: 100nF, APRLPrints:C_0603
- removed C100, C111, C112, C123, C124, C135, C136, C75, C76, C87, C88, C99: 22nF, APRLPrints:C_0603
- removed C102, C104, C106, C108, C114, C116, C118, C120, C126, C128, C130, C132, C138, C140, C142, C144, C78, C8, C80, C82, C84, C90, C92, C94, C96: 470pF, APRLPrints:C_0603
- removed C105, C107, C117, C119, C129, C131, C141, C143, C81, C83, C93, C95: 100uF, Capacitor_SMD:CP_Elec_10x10.5
- removed C110, C122, C134, C47, C48, C74, C86, C98: 2.2uF, APRLPrints:C_0603
- removed C12, C14, C2, C4, C51, C52: 10pF, APRLPrints:C_0603
- removed C13, C15, C22, C24, C25, C28, C31, C34, C41, C42, C43, C44, C45, C46: 22uF, APRLPrints:C_0805
- removed C53, C55, C58, C60, C63, C65, C68, C70: 10n, APRLPrints:C_0603
- removed C54, C56, C57, C59, C61, C62, C64, C66, C67, C69, C71, C72: 100n, APRLPrints:C_0603
- removed C9: 220nF, APRLPrints:C_0603
- removed D1, D10, D14, D20, D21, D24, D25, D28, D3, D30, D32, D34, D36, D5, D6, D7: LED_Small, APRLPrints:LED_0603
- removed D11, D13, D15, D22, D23, D26, D27, D29, D31, D33, D35, D37, D8, D9: SS54, Diode_SMD:D_SMA
- removed D16, D17, D18, D19: LED, APRLPrints:LED_0603
- removed D2, D4: PMEG3010BER, Diode_SMD:Nexperia_CFP3_SOD-123W
- removed F1, F2: 500mA, Fuse:Fuse_0805_2012Metric
- removed F3, F6: XF-508P-B-B, Fuse:Fuseholder_Blade_Mini_Keystone_3568
- removed F4: XFCN XF-508P-B-B, Fuse:Fuseholder_Blade_Mini_Keystone_3568
- removed J1: Conn_02x05_Odd_Even, Connector_PinHeader_2.54mm:PinHeader_1x10_P2.54mm_Vertical
- removed J10, J27, J28, J29, J30, J41, J42, J43, J44, J45: Conn_01x02, Connector_Molex:Molex_Micro-Fit_3.0_43650-0215_1x02_P3.00mm_Vertical
- removed J11, J12, J13, J14, J15, J16, J17, J18, J19, J20, J21, J22, J23, J24, J25, J26: Conn_01x03, Connector_Molex:Molex_Micro-Fit_3.0_43650-0315_1x03_P3.00mm_Vertical
- removed J2, J4: USB_C_Receptacle_USB2.0_16P, Connector_USB:USB_C_Receptacle_HRO_TYPE-C-31-M-12
- removed J3: RJ45_Hanrun_HR911105A_Horizontal, Connector_RJ:RJ45_Hanrun_HR911105A_Horizontal
- removed J31, J32, J33, J34, J35, J36: Conn_01x04, Connector_JST:JST_XH_B4B-XH-AM_1x04_P2.50mm_Vertical
- removed J37, J38, J39, J40, J6, J7, J9: Screw_Terminal_01x02, Connector_Phoenix_MSTB:PhoenixContact_MSTBA_2,5_2-G_1x02_P5.00mm_Horizontal
- removed J5: Conn_02x05_Odd_Even, Connector_PinHeader_2.54mm:PinHeader_2x05_P2.54mm_Vertical
- removed L1: 3.3 uH, Inductor_SMD:L_1008_2520Metric
- removed Q1, Q10, Q6, Q7, Q8, Q9: AO3400A, Package_TO_SOT_SMD:SOT-23
- removed Q2, Q3, Q4, Q5: Si7450DP, Package_SO:PowerPAK_SO-8_Single
- removed R1, R12, R16, R17, R18, R19, R21, R23, R25, R27, R28, R29, R3, R30, R31, R32, R33, R34, R35, R36, R37, R38, R39, R40, R41, R42, R43, R44, R45, R46, R47, R48, R49, R50, R61, R62, R67, R68, R70, R73, R76, R79, R82: 10k, APRLPrints:R_0603
- removed R10, R14, R15, R9: 4.7k, APRLPrints:R_0603
- removed R11, R13: 330R, APRLPrints:R_0603
- removed R2, R20: 1.5k, APRLPrints:R_0603
- removed R22: 56.2k, APRLPrints:R_0603
- removed R24, R57, R58, R63, R64, R69, R72, R75, R78, R81: 10R, APRLPrints:R_0603
- removed R26, R59, R60, R65, R66, R71, R74, R77, R80, R83: 100k, APRLPrints:R_0603
- removed R4, R5, R7, R8: 47R, APRLPrints:R_0603
- removed R51, R52, R53, R54, R55, R56: 24k, APRLPrints:R_0603
- removed R6: 12.1k, APRLPrints:R_0603
- removed SW1, SW2: SKRPANE010, APRLPrints:SKRPANE010
- removed U1: STM32H723ZGT6, Package_QFP:LQFP-144_20x20mm_P0.5mm
- removed U10, U11, U12, U9: LTV-247, Package_SO:SOP-16_4.4x10.4mm_P1.27mm
- removed U13, U14, U15, U16: MAX31856, Package_SO:TSSOP-14_4.4x5mm_P0.65mm
- removed U17, U18, U19, U20, U21, U22: TMC2241ATC, libserie:QFN-38_EP_5.63x7.6_Pitch0.5mm
- removed U2: LAN8742A, Package_DFN_QFN:VQFN-24-1EP_4x4mm_P0.5mm_EP2.5x2.5mm_ThermalVias
- removed U23, U24: UCC27524DGN, Package_SO:Texas_DGN0008G_VSSOP-8-1EP_3x3mm_P0.65mm_EP2x2.94mm_Mask1.846x2.15mm_ThermalVias
- removed U3, U4: USBLC6-2SC6, Package_TO_SOT_SMD:SOT-23-6
- removed U5, U8: AP2112K-3.3, Package_TO_SOT_SMD:SOT-23-5
- removed U6: STM32F103C8Tx, Package_QFP:LQFP-48_7x7mm_P0.5mm
- removed U7: AP62300TWU, Package_TO_SOT_SMD:TSOT-23-6
- removed Y1, Y3: 25 MHz, APRLPrints:3225-4P-L
- removed Y2: 8 MHz, APRLPrints:3225-4P-L
Routing:
- net /Connections/High Power Outputs 1/High Power Output Set 2/OUTB: track 7.19 -> 0.00 mm
- net /Connections/High Power Outputs 1/High Power Output Set 1/OUTA: track 4.60 -> 0.00 mm
- net /Connections/High Power Outputs 1/High Power Output Set 2/OUTA: track 4.50 -> 0.00 mm
- net Net-(J9-Pin_2): vias 44 -> 0
- net GND: vias 116 -> 0
- removed copper zone on B.Cu, net /Connections/High Power Outputs 1/High Power Output Set 1/PWR
- removed copper zone on F.Cu, net /Connections/High Power Outputs 1/High Power Output Set 1/PWR
- removed copper zone on In1.Cu, net /Connections/High Power Outputs 1/High Power Output Set 1/PWR
- removed copper zone on In2.Cu, net /Connections/High Power Outputs 1/High Power Output Set 1/PWR
- removed copper zone on F.Cu, net GND
- removed copper zone on B.Cu, net Net-(D24-K)
- removed copper zone on F.Cu, net Net-(D24-K)
- removed copper zone on In1.Cu, net Net-(D24-K)
- removed copper zone on In2.Cu, net Net-(D24-K)
- removed copper zone on B.Cu, net Net-(D25-K)
- removed copper zone on F.Cu, net Net-(D25-K)
- removed copper zone on In1.Cu, net Net-(D25-K)
- removed copper zone on In2.Cu, net Net-(D25-K)
- removed copper zone on B.Cu, net Net-(J9-Pin_2)
- removed copper zone on F.Cu, net Net-(J9-Pin_2)
- removed copper zone on In1.Cu, net Net-(J9-Pin_2)
- removed copper zone on In2.Cu, net Net-(J9-Pin_2)
Other:
- board outline removed

Commit message: loadcell math coming soon(tm)
Parts:
- added C1: 2.2uF, APRLPrints:C_0603, F.Cu at (-71.8, 54.5)
- added C100: 100uF, Capacitor_SMD:CP_Elec_10x10.5, F.Cu at (-60.6, 71.4)
- added C101: 470pF, APRLPrints:C_0603, F.Cu at (-44.6, 64.8)
- added C102: 100nF, APRLPrints:C_0603, F.Cu at (-86.2, 93.1)
- added C103: 2.2uF, APRLPrints:C_0603, F.Cu at (-86.2, 95.5)
- added C104: 22nF, APRLPrints:C_0603, F.Cu at (-86.2, 98.0)
- added C105: 22nF, APRLPrints:C_0603, F.Cu at (-86.2, 100.4)
- added C106: 100nF, APRLPrints:C_0603, F.Cu at (-82.6, 93.1)
- added C107: 470pF, APRLPrints:C_0603, F.Cu at (-82.6, 95.5)
- added C108: 100nF, APRLPrints:C_0603, F.Cu at (-82.6, 98.0)
- added C109: 470pF, APRLPrints:C_0603, F.Cu at (-82.6, 100.4)
- added C110: 100uF, Capacitor_SMD:CP_Elec_10x10.5, F.Cu at (94.2, 27.6)
- added C111: 470pF, APRLPrints:C_0603, F.Cu at (-79.1, 93.1)
- added C112: 100uF, Capacitor_SMD:CP_Elec_10x10.5, F.Cu at (94.4, 38.8)
- added C113: 470pF, APRLPrints:C_0603, F.Cu at (-79.1, 95.5)
- added C114: 100nF, APRLPrints:C_0603, F.Cu at (-55.1, 122.5)
- added C115: 2.2uF, APRLPrints:C_0603, F.Cu at (-55.1, 125.0)
- added C116: 22nF, APRLPrints:C_0603, F.Cu at (-55.1, 127.4)
- added C117: 22nF, APRLPrints:C_0603, F.Cu at (-55.1, 129.9)
- added C118: 100nF, APRLPrints:C_0603, F.Cu at (-51.6, 122.5)
- added C119: 470pF, APRLPrints:C_0603, F.Cu at (-51.6, 125.0)
- added C120: 100nF, APRLPrints:C_0603, F.Cu at (-51.6, 127.4)
- added C121: 470pF, APRLPrints:C_0603, F.Cu at (-51.6, 129.9)
- added C122: 100uF, Capacitor_SMD:CP_Elec_10x10.5, F.Cu at (-64.1, 119.5)
- added C123: 470pF, APRLPrints:C_0603, F.Cu at (-48.0, 122.5)
- added C124: 100uF, Capacitor_SMD:CP_Elec_10x10.5, F.Cu at (-64.1, 131.6)
- added C125: 470pF, APRLPrints:C_0603, F.Cu at (-48.0, 125.0)
- added C126: 100nF, APRLPrints:C_0603, F.Cu at (-86.2, 122.5)
- added C127: 2.2uF, APRLPrints:C_0603, F.Cu at (-86.2, 125.0)
- added C128: 22nF, APRLPrints:C_0603, F.Cu at (-86.2, 127.4)
- added C129: 22nF, APRLPrints:C_0603, F.Cu at (-86.2, 129.9)
- added C130: 100nF, APRLPrints:C_0603, F.Cu at (-82.6, 122.5)
- added C131: 470pF, APRLPrints:C_0603, F.Cu at (-82.6, 125.0)
- added C132: 100nF, APRLPrints:C_0603, F.Cu at (-82.6, 127.4)
- added C133: 470pF, APRLPrints:C_0603, F.Cu at (-82.6, 129.9)
- added C134: 100uF, Capacitor_SMD:CP_Elec_10x10.5, F.Cu at (-95.1, 119.5)
- added C135: 470pF, APRLPrints:C_0603, F.Cu at (-79.1, 122.5)
- added C136: 100uF, Capacitor_SMD:CP_Elec_10x10.5, F.Cu at (-95.1, 131.6)
- added C137: 470pF, APRLPrints:C_0603, F.Cu at (-79.1, 125.0)
- added C138: 100nF, APRLPrints:C_0603, F.Cu at (-24.1, 93.1)
- added C139: 2.2uF, APRLPrints:C_0603, F.Cu at (-24.1, 95.5)
- added C140: 22nF, APRLPrints:C_0603, F.Cu at (-24.1, 98.0)
- added C141: 22nF, APRLPrints:C_0603, F.Cu at (-24.1, 100.4)
- added C142: 100nF, APRLPrints:C_0603, F.Cu at (-20.6, 93.1)
- added C143: 470pF, APRLPrints:C_0603, F.Cu at (-20.6, 95.5)
- added C144: 100nF, APRLPrints:C_0603, F.Cu at (-20.6, 98.0)
- added C145: 470pF, APRLPrints:C_0603, F.Cu at (-20.6, 100.4)
- added C146: 100uF, Capacitor_SMD:CP_Elec_10x10.5, F.Cu at (-33.1, 90.1)
- added C147: 470pF, APRLPrints:C_0603, F.Cu at (-17.0, 93.1)
- added C148: 100uF, Capacitor_SMD:CP_Elec_10x10.5, F.Cu at (-33.1, 102.1)
- added C149: 470pF, APRLPrints:C_0603, F.Cu at (-17.0, 95.5)
- added C2: 2.2uF, APRLPrints:C_0603, F.Cu at (-71.8, 57.0)
- added C21: 100nF, APRLPrints:C_0603, F.Cu at (-24.6, 132.6)
- added C23: 100nF, APRLPrints:C_0603, F.Cu at (-24.6, 135.0)
- added C28: 100nF, APRLPrints:C_0603, F.Cu at (-117.0, 69.3)
- added C29: 100nF, APRLPrints:C_0603, F.Cu at (-117.0, 71.8)
- added C3: 100nF, APRLPrints:C_0603, F.Cu at (-71.8, 59.5)
- added C30: 100nF, APRLPrints:C_0603, F.Cu at (-117.0, 74.2)
- added C31: 100nF, APRLPrints:C_0603, F.Cu at (-117.0, 76.7)
- added C32: 22uF, APRLPrints:C_0805, F.Cu at (-137.1, 35.6)
- added C33: 22uF, APRLPrints:C_0805, F.Cu at (-137.1, 38.5)
- added C34: 22uF, APRLPrints:C_0805, F.Cu at (-137.1, 41.4)
- added C39: 22uF, APRLPrints:C_0805, F.Cu at (-137.1, 44.2)
- added C4: 10pF, APRLPrints:C_0603, F.Cu at (-71.8, 61.9)
- added C42: 22uF, APRLPrints:C_0805, F.Cu at (-137.1, 47.0)
- added C43: 22uF, APRLPrints:C_0805, F.Cu at (-137.1, 49.9)
- added C46: 100nF, APRLPrints:C_0603, F.Cu at (-133.3, 35.5)
- added C47: 100nF, APRLPrints:C_0603, F.Cu at (-133.3, 37.9)
- added C48: 100nF, APRLPrints:C_0603, F.Cu at (-133.3, 40.4)
- added C5: 10pF, APRLPrints:C_0603, F.Cu at (-71.8, 64.3)
- added C51: 100nF, APRLPrints:C_0603, F.Cu at (-133.3, 42.8)
- added C52: 100nF, APRLPrints:C_0603, F.Cu at (-133.3, 45.2)
- added C55: 100nF, APRLPrints:C_0603, F.Cu at (-133.3, 47.7)
- added C58: 100nF, APRLPrints:C_0603, F.Cu at (-129.7, 35.5)
- added C62: 100nF, APRLPrints:C_0603, F.Cu at (-129.7, 37.9)
- added C63: 100nF, APRLPrints:C_0603, F.Cu at (-129.7, 40.4)
- added C64: 100nF, APRLPrints:C_0603, F.Cu at (-129.7, 42.8)
- added C66: 100nF, APRLPrints:C_0603, F.Cu at (-129.7, 45.2)
- added C67: 100nF, APRLPrints:C_0603, F.Cu at (-129.7, 47.7)
- added C68: 100nF, APRLPrints:C_0603, F.Cu at (-128.7, 85.5)
- added C69: 1uF, APRLPrints:C_0603, F.Cu at (-128.7, 88.0)
- added C70: 100nF, APRLPrints:C_0603, F.Cu at (-35.2, 54.5)
- added C71: 1uF, APRLPrints:C_0603, F.Cu at (-35.2, 57.0)
- added C72: 10nF, APRLPrints:C_0603, F.Cu at (-155.0, 121.1)
- added C73: 100nF, APRLPrints:C_0603, F.Cu at (-155.0, 123.6)
- added C74: 100nF, APRLPrints:C_0603, F.Cu at (-155.0, 126.0)
- added C75: 10nF, APRLPrints:C_0603, F.Cu at (-25.5, 17.1)
- added C76: 100nF, APRLPrints:C_0603, F.Cu at (-25.5, 19.6)
- added C77: 100nF, APRLPrints:C_0603, F.Cu at (-25.5, 22.0)
- added C78: 100nF, APRLPrints:C_0603, F.Cu at (-55.1, 93.1)
- added C79: 2.2uF, APRLPrints:C_0603, F.Cu at (-55.1, 95.5)
- added C80: 22nF, APRLPrints:C_0603, F.Cu at (-55.1, 98.0)
- added C81: 22nF, APRLPrints:C_0603, F.Cu at (-55.1, 100.4)
- added C82: 100nF, APRLPrints:C_0603, F.Cu at (-51.6, 93.1)
- added C83: 470pF, APRLPrints:C_0603, F.Cu at (-51.6, 95.5)
- added C84: 100nF, APRLPrints:C_0603, F.Cu at (-51.6, 98.0)
- added C85: 470pF, APRLPrints:C_0603, F.Cu at (-51.6, 100.4)
- added C86: 100uF, Capacitor_SMD:CP_Elec_10x10.5, F.Cu at (-64.1, 90.1)
- added C87: 470pF, APRLPrints:C_0603, F.Cu at (-48.0, 93.1)
- added C88: 100uF, Capacitor_SMD:CP_Elec_10x10.5, F.Cu at (-64.1, 102.1)
- added C89: 470pF, APRLPrints:C_0603, F.Cu at (-48.0, 95.5)
- added C90: 100nF, APRLPrints:C_0603, F.Cu at (-51.7, 62.4)
- added C91: 2.2uF, APRLPrints:C_0603, F.Cu at (-51.7, 64.8)
- added C92: 22nF, APRLPrints:C_0603, F.Cu at (-51.7, 67.2)
- added C93: 22nF, APRLPrints:C_0603, F.Cu at (-51.7, 69.7)
- added C94: 100nF, APRLPrints:C_0603, F.Cu at (-48.1, 62.4)
- added C95: 470pF, APRLPrints:C_0603, F.Cu at (-48.1, 64.8)
- added C96: 100nF, APRLPrints:C_0603, F.Cu at (-48.1, 67.2)
- added C97: 470pF, APRLPrints:C_0603, F.Cu at (-48.1, 69.7)
- added C98: 100uF, Capacitor_SMD:CP_Elec_10x10.5, F.Cu at (-60.6, 59.4)
- added C99: 470pF, APRLPrints:C_0603, F.Cu at (-44.6, 62.4)
- added D1: LED_Small, APRLPrints:LED_0603, F.Cu at (-106.3, 69.4)
- added D10: LED_Small, APRLPrints:LED_0603, F.Cu at (-114.5, 49.8)
- added D11: LED_Small, APRLPrints:LED_0603, F.Cu at (-117.7, 99.0)
- added D12: LED_Small, APRLPrints:LED_0603, F.Cu at (-117.7, 101.6)
- added D13: LED_Small, APRLPrints:LED_0603, F.Cu at (-24.2, 68.0)
- added D14: LED_Small, APRLPrints:LED_0603, F.Cu at (-24.2, 70.6)
- added D15: LED_Small, APRLPrints:LED_0603, F.Cu at (-111.4, 119.5)
- added D16: LED_Small, APRLPrints:LED_0603, F.Cu at (-125.1, 136.7)
- added D17: LED_Small, APRLPrints:LED_0603, F.Cu at (-125.1, 119.5)
- added D18: LED, APRLPrints:LED_0603, F.Cu at (-143.7, 129.0)
- added D19: LED, APRLPrints:LED_0603, F.Cu at (-14.2, 25.0)
- added D2: PMEG3010BER, Diode_SMD:Nexperia_CFP3_SOD-123W, F.Cu at (-116.0, 79.5)
- added D3: LED_Small, APRLPrints:LED_0603, F.Cu at (-106.3, 72.0)
- added D4: LED_Small, APRLPrints:LED_0603, F.Cu at (-106.3, 74.6)
- added D5: LED_Small, APRLPrints:LED_0603, F.Cu at (-106.3, 77.2)
- added D6: SS54, Diode_SMD:D_SMA, F.Cu at (-112.3, 36.5)
- added D7: LED_Small, APRLPrints:LED_0603, F.Cu at (-114.5, 44.6)
- added D8: SS54, Diode_SMD:D_SMA, F.Cu at (-112.3, 41.0)
- added D9: LED_Small, APRLPrints:LED_0603, F.Cu at (-114.5, 47.2)
- added F1: 500mA, Fuse:Fuse_0805_2012Metric, F.Cu at (-111.0, 79.3)
- added F2: XFCN XF-508P-B-B, Fuse:Fuseholder_Blade_Mini_Keystone_3568, F.Cu at (-152.9, 36.7)
- added F3: XF-508P-B-B, Fuse:Fuseholder_Blade_Mini_Keystone_3568, F.Cu at (-152.9, 45.0)
- added H1: MountingHole, MountingHole:MountingHole_3.2mm_M3, F.Cu at (-33.2, 19.9)
- added H2: MountingHole, MountingHole:MountingHole_3.2mm_M3, F.Cu at (-33.2, 27.8)
- added H3: MountingHole, MountingHole:MountingHole_3.2mm_M3, F.Cu at (-33.2, 35.8)
- added H4: MountingHole, MountingHole:MountingHole_3.2mm_M3, F.Cu at (-33.2, 43.7)
- added J1: Conn_02x05_Odd_Even, Connector_PinHeader_2.54mm:PinHeader_1x10_P2.54mm_Vertical, F.Cu at (-100.2, 55.6)
- added J10: Screw_Terminal_01x02, Connector_Phoenix_MSTB:PhoenixContact_MSTBA_2,5_2-G_1x02_P5.00mm_Horizontal, F.Cu at (-36.0, 117.0)
- added J11: USB_C_Receptacle_USB2.0_16P, Connector_USB:USB_C_Receptacle_HRO_TYPE-C-31-M-12, F.Cu at (-124.7, 59.1)
- added J12: USB_C_Receptacle_USB2.0_16P, Connector_USB:USB_C_Receptacle_HRO_TYPE-C-31-M-12, F.Cu at (-124.7, 69.6)
- added J13: Conn_02x05_Odd_Even, Connector_PinHeader_2.54mm:PinHeader_2x05_P2.54mm_Vertical, F.Cu at (-116.5, 55.6)
- added J14: Screw_Terminal_06x01x02, TerminalBlock_Ningbo-Kagnex:TerminalBlock_Ningbo-Kagnex_HB9500M_1x12_P9.5mm, F.Cu at (85.2, 155.7)
- added J15: Conn_01x02, Connector_Molex:Molex_Micro-Fit_3.0_43650-0215_1x02_P3.00mm_Vertical, F.Cu at (-19.4, 19.4)
- added J16: Conn_01x02, Connector_Molex:Molex_Micro-Fit_3.0_43650-0215_1x02_P3.00mm_Vertical, F.Cu at (-112.4, 109.4)
- added J17: Conn_01x02, Connector_Molex:Molex_Micro-Fit_3.0_43650-0215_1x02_P3.00mm_Vertical, F.Cu at (-126.1, 126.6)
- added J18: Conn_01x02, Connector_Molex:Molex_Micro-Fit_3.0_43650-0215_1x02_P3.00mm_Vertical, F.Cu at (-126.1, 109.4)
- added J19: Conn_01x03, Connector_Molex:Molex_Micro-Fit_3.0_43650-0315_1x03_P3.00mm_Vertical, F.Cu at (-152.4, 90.1)
- added J20: Conn_01x03, Connector_Molex:Molex_Micro-Fit_3.0_43650-0315_1x03_P3.00mm_Vertical, F.Cu at (-152.4, 97.9)
- added J21: Conn_01x03, Connector_Molex:Molex_Micro-Fit_3.0_43650-0315_1x03_P3.00mm_Vertical, F.Cu at (-152.4, 105.7)
- added J22: Conn_01x03, Connector_Molex:Molex_Micro-Fit_3.0_43650-0315_1x03_P3.00mm_Vertical, F.Cu at (-152.4, 113.6)
- added J23: Conn_01x03, Connector_Molex:Molex_Micro-Fit_3.0_43650-0315_1x03_P3.00mm_Vertical, F.Cu at (-152.4, 56.8)
- added J24: Conn_01x03, Connector_Molex:Molex_Micro-Fit_3.0_43650-0315_1x03_P3.00mm_Vertical, F.Cu at (-152.4, 64.6)
- added J25: Conn_01x03, Connector_Molex:Molex_Micro-Fit_3.0_43650-0315_1x03_P3.00mm_Vertical, F.Cu at (-152.4, 72.5)
- added J26: Conn_01x03, Connector_Molex:Molex_Micro-Fit_3.0_43650-0315_1x03_P3.00mm_Vertical, F.Cu at (-152.4, 80.3)
- added J27: Conn_01x02, Connector_Molex:Molex_Micro-Fit_3.0_43650-0215_1x02_P3.00mm_Vertical, F.Cu at (-148.8, 123.4)
- added J29: Conn_01x04, Connector_JST:JST_XH_B4B-XH-AM_1x04_P2.50mm_Vertical, F.Cu at (-53.5, 87.4)
- added J30: Conn_01x04, Connector_JST:JST_XH_B4B-XH-AM_1x04_P2.50mm_Vertical, F.Cu at (-50.0, 56.7)
- added J31: Conn_01x04, Connector_JST:JST_XH_B4B-XH-AM_1x04_P2.50mm_Vertical, F.Cu at (-84.5, 87.4)
- added J32: Conn_01x04, Connector_JST:JST_XH_B4B-XH-AM_1x04_P2.50mm_Vertical, F.Cu at (-53.5, 116.9)
- added J33: Conn_01x04, Connector_JST:JST_XH_B4B-XH-AM_1x04_P2.50mm_Vertical, F.Cu at (101.7, 16.8)
- added J34: Conn_01x04, Connector_JST:JST_XH_B4B-XH-AM_1x04_P2.50mm_Vertical, F.Cu at (-22.4, 87.4)
- added Q1: CSD18532NQ5B, Package_TO_SOT_SMD:TDSON-8-1, F.Cu at (-122.8, 87.7)
- added Q2: CSD18532NQ5B, Package_TO_SOT_SMD:TDSON-8-1, F.Cu at (-122.8, 94.4)
- added Q3: CSD18532NQ5B, Package_TO_SOT_SMD:TDSON-8-1, F.Cu at (-29.4, 56.7)
- added Q4: CSD18532NQ5B, Package_TO_SOT_SMD:TDSON-8-1, F.Cu at (-29.4, 63.4)
- added Q5: AO3400A, Package_TO_SOT_SMD:SOT-23, F.Cu at (-110.8, 116.0)
- added Q6: AO3400A, Package_TO_SOT_SMD:SOT-23, F.Cu at (-124.5, 133.1)
- added Q7: AO3400A, Package_TO_SOT_SMD:SOT-23, F.Cu at (-124.5, 116.0)
- added R22: 4.7k, APRLPrints:R_0603, F.Cu at (-113.5, 69.3)
- added R23: 4.7k, APRLPrints:R_0603, F.Cu at (-113.5, 71.8)
- added R24: 4.7k, APRLPrints:R_0603, F.Cu at (-113.5, 74.2)
- added R25: 4.7k, APRLPrints:R_0603, F.Cu at (-113.5, 76.7)
- added R26: 10k, APRLPrints:R_0603, F.Cu at (-109.9, 69.3)
- added R27: 10k, APRLPrints:R_0603, F.Cu at (-109.9, 71.8)
- added R28: 10k, APRLPrints:R_0603, F.Cu at (-109.9, 74.2)
- added R29: 10k, APRLPrints:R_0603, F.Cu at (-109.9, 76.7)
- added R34: 10k, APRLPrints:R_0603, F.Cu at (-126.2, 35.5)
- added R39: 10k, APRLPrints:R_0603, F.Cu at (-126.2, 37.9)
- added R40: 10k, APRLPrints:R_0603, F.Cu at (-126.2, 40.4)
- added R41: 10R, APRLPrints:R_0603, F.Cu at (-128.7, 90.4)
- added R42: 10R, APRLPrints:R_0603, F.Cu at (-128.7, 92.9)
- added R43: 100k, APRLPrints:R_0603, F.Cu at (-128.7, 95.3)
- added R44: 100k, APRLPrints:R_0603, F.Cu at (-128.7, 97.8)
- added R45: 10k, APRLPrints:R_0603, F.Cu at (-128.7, 100.2)
- added R46: 10k, APRLPrints:R_0603, F.Cu at (-128.7, 102.7)
- added R47: 10R, APRLPrints:R_0603, F.Cu at (-35.2, 59.5)
- added R48: 10R, APRLPrints:R_0603, F.Cu at (-35.2, 61.9)
- added R49: 100k, APRLPrints:R_0603, F.Cu at (-35.2, 64.3)
- added R50: 100k, APRLPrints:R_0603, F.Cu at (-35.2, 66.8)
- added R51: 10k, APRLPrints:R_0603, F.Cu at (-35.2, 69.2)
- added R52: 10k, APRLPrints:R_0603, F.Cu at (-35.2, 71.7)
- added R53: 10R, APRLPrints:R_0603, F.Cu at (-115.0, 115.0)
- added R54: 10k, APRLPrints:R_0603, F.Cu at (-115.0, 117.4)
- added R55: 100k, APRLPrints:R_0603, F.Cu at (-115.0, 119.9)
- added R56: 10R, APRLPrints:R_0603, F.Cu at (-128.7, 132.1)
- added R57: 10k, APRLPrints:R_0603, F.Cu at (-128.7, 134.6)
- added R58: 100k, APRLPrints:R_0603, F.Cu at (-128.7, 137.0)
- added R59: 10R, APRLPrints:R_0603, F.Cu at (-128.7, 115.0)
- added R60: 10k, APRLPrints:R_0603, F.Cu at (-128.7, 117.4)
- added R61: 100k, APRLPrints:R_0603, F.Cu at (-128.7, 119.9)
- added R62: 10k, APRLPrints:R_0603, F.Cu at (-140.3, 99.9)
- added R63: 10k, APRLPrints:R_0603, F.Cu at (-140.3, 102.3)
- added R64: 10k, APRLPrints:R_0603, F.Cu at (-140.3, 104.8)
- added R65: 10k, APRLPrints:R_0603, F.Cu at (-140.3, 107.2)
- added R66: 10k, APRLPrints:R_0603, F.Cu at (-140.3, 66.6)
- added R67: 10k, APRLPrints:R_0603, F.Cu at (-140.3, 69.0)
- added R68: 10k, APRLPrints:R_0603, F.Cu at (-140.3, 71.5)
- added R69: 10k, APRLPrints:R_0603, F.Cu at (-140.3, 73.9)
- added R70: 4.02k, APRLPrints:R_0603, F.Cu at (-155.0, 128.5)
- added R71: 10k, APRLPrints:R_0603, F.Cu at (-155.0, 130.9)
- added R72: 10k, APRLPrints:R_0603, F.Cu at (-155.0, 133.4)
- added R73: 4.02k, APRLPrints:R_0603, F.Cu at (-25.5, 24.5)
- added R74: 10k, APRLPrints:R_0603, F.Cu at (-25.5, 26.9)
- added R75: 10k, APRLPrints:R_0603, F.Cu at (-25.5, 29.4)
- added R76: 24k, APRLPrints:R_0603, F.Cu at (-48.0, 98.0)
- added R77: 24k, APRLPrints:R_0603, F.Cu at (-44.6, 67.2)
- added R78: 24k, APRLPrints:R_0603, F.Cu at (-79.1, 98.0)
- added R79: 24k, APRLPrints:R_0603, F.Cu at (-48.0, 127.4)
- added R80: 24k, APRLPrints:R_0603, F.Cu at (-79.1, 127.4)
- added R81: 24k, APRLPrints:R_0603, F.Cu at (-17.0, 98.0)
- added SW1: SKRPANE010, APRLPrints:SKRPANE010, F.Cu at (-94.6, 79.8)
- added SW2: SKRPANE010, APRLPrints:SKRPANE010, F.Cu at (-108.3, 64.7)
- added U1: STM32H723ZGT6, Package_QFP:LQFP-144_20x20mm_P0.5mm, F.Cu at (-85.8, 65.5)
- added U11: USBLC6-2SC6, Package_TO_SOT_SMD:SOT-23-6, F.Cu at (-109.1, 55.7)
- added U12: USBLC6-2SC6, Package_TO_SOT_SMD:SOT-23-6, F.Cu at (-109.1, 60.4)
- added U13: STM32F042F4Px, Package_SO:TSSOP-20_4.4x6.5mm_P0.65mm, F.Cu at (-125.7, 78.3)
- added U14: AP2112K-3.3, Package_TO_SOT_SMD:SOT-23-5, F.Cu at (-105.7, 36.6)
- added U15: AP64500, Package_SO:Diodes_SO-8EP, F.Cu at (-120.4, 37.7)
- added U16: AP64500, Package_SO:Diodes_SO-8EP, F.Cu at (-120.4, 44.3)
- added U17: TPS7A20xxxDQN, Package_SON:Texas_X2SON-4_1x1mm_P0.65mm, F.Cu at (-106.6, 40.1)
- added U18: UCC27524DGN, Package_SO:Texas_DGN0008G_VSSOP-8-1EP_3x3mm_P0.65mm_EP2x2.94mm_Mask1.846x2.15mm_ThermalVias, F.Cu at (-123.2, 100.1)
- added U19: UCC27524DGN, Package_SO:Texas_DGN0008G_VSSOP-8-1EP_3x3mm_P0.65mm_EP2x2.94mm_Mask1.846x2.15mm_ThermalVias, F.Cu at (-29.8, 69.1)
- added U20: LTV-247, Package_SO:SOP-16_4.4x10.4mm_P1.27mm, F.Cu at (-137.3, 92.7)
- added U21: LTV-247, Package_SO:SOP-16_4.4x10.4mm_P1.27mm, F.Cu at (-137.3, 59.4)
- added U22: MAX31865xTP, Package_DFN_QFN:TQFN-20-1EP_5x5mm_P0.65mm_EP3.25x3.25mm, F.Cu at (-149.2, 131.3)
- added U23: MAX31865xTP, Package_DFN_QFN:TQFN-20-1EP_5x5mm_P0.65mm_EP3.25x3.25mm, F.Cu at (-19.7, 27.4)
- added U24: TMC2241ATC, libserie:QFN-38_EP_5.63x7.6_Pitch0.5mm, F.Cu at (104.5, 33.6)
- added U25: TMC2241ATC, libserie:QFN-38_EP_5.63x7.6_Pitch0.5mm, F.Cu at (-49.5, 75.8)
- added U26: TMC2241ATC, libserie:QFN-38_EP_5.63x7.6_Pitch0.5mm, F.Cu at (-84.0, 106.6)
- added U27: TMC2241ATC, libserie:QFN-38_EP_5.63x7.6_Pitch0.5mm, F.Cu at (-53.0, 136.0)
- added U28: TMC2241ATC, libserie:QFN-38_EP_5.63x7.6_Pitch0.5mm, F.Cu at (-84.0, 136.0)
- added U29: TMC2241ATC, libserie:QFN-38_EP_5.63x7.6_Pitch0.5mm, F.Cu at (-21.9, 106.6)
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