File: Serie.kicad_pcb (KiCad board)
At the start: 4 copper layers, 249 parts, among them J1 Conn_02x05_Odd_Even, J10 Screw_Terminal_01x02, J11 USB_C_Receptacle_USB2.0_16P, J12 USB_C_Receptacle_USB2.0_16P, J13 Conn_02x05_Odd_Even, J14 Screw_Terminal_06x01x02, J15 Conn_01x02, J16 Conn_01x02, J17 Conn_01x02, J18 Conn_01x02, J19 Conn_01x03, J20 Conn_01x03, J21 Conn_01x03, J22 Conn_01x03, J23 Conn_01x03, J24 Conn_01x03, J25 Conn_01x03, J26 Conn_01x03, J27 Conn_01x02, J29 Conn_01x04, J30 Conn_01x04, J31 Conn_01x04, J32 Conn_01x04, J33 Conn_01x04, J34 Conn_01x04, Q1 CSD18532NQ5B, Q2 CSD18532NQ5B, Q3 CSD18532NQ5B, Q4 CSD18532NQ5B, Q5 AO3400A, Q6 AO3400A, Q7 AO3400A, SW1 SKRPANE010, SW2 SKRPANE010, U1 STM32H723ZGT6, U11 USBLC6-2SC6, U12 USBLC6-2SC6, U13 STM32F042F4Px, U14 AP2112K-3.3, U15 AP64500, U16 AP64500, U17 TPS7A20xxxDQN, U18 UCC27524DGN, U19 UCC27524DGN, U20 LTV-247, U21 LTV-247, U22 MAX31865xTP, U23 MAX31865xTP, U24 TMC2241ATC, U25 TMC2241ATC, U26 TMC2241ATC, U27 TMC2241ATC, U28 TMC2241ATC, U29 TMC2241ATC, U4 LDC1612, U5 ADS1115IDGS, U6 ADS1220xPW, U8 TMUX1101DBV, U9 TMUX1108PW, Y1 25 MHz

Commit message: a
Parts:
- added ?: , , F.Cu at (97.5, 123.5)
- added ?: , , F.Cu at (104.5, 140.5)
- added ?: , , F.Cu at (101.5, 149.0)
- added ?: , , F.Cu at (118.5, 100.5)
- added ?: , , F.Cu at (104.5, 145.5)
- added ?: , , F.Cu at (124.0, 74.0)
- added ?: , , F.Cu at (214.0, 153.5)
- added ?: , , F.Cu at (100.0, 123.5)
- added ?: , , F.Cu at (105.5, 107.5)
- added ?: , , F.Cu at (96.5, 149.0)
- added ?: , , F.Cu at (98.7, 113.1)
- added ?: , , F.Cu at (113.5, 100.5)
- added ?: , , F.Cu at (211.5, 153.5)
- added ?: , , F.Cu at (104.5, 127.5)
- added ?: , , F.Cu at (124.0, 76.5)
- added ?: , , F.Cu at (101.2, 113.1)
- added ?: , , F.Cu at (95.0, 123.5)
- added ?: , , F.Cu at (216.5, 153.5)
- added ?: , , F.Cu at (103.7, 113.1)
- added ?: , , F.Cu at (105.5, 110.0)
- added ?: , , F.Cu at (104.5, 122.5)
- added ?: , , F.Cu at (124.0, 71.5)
- added ?: , , F.Cu at (104.5, 143.0)
- added ?: , , F.Cu at (105.5, 105.0)
- added ?: , , F.Cu at (116.0, 100.5)
- added ?: , , F.Cu at (99.0, 149.0)
- added ?: , , F.Cu at (104.5, 125.0)
- added C10: 10uF, APRLPrints:C_0603, B.Cu at (32.3, 24.9)
- added C11: 10nF, APRLPrints:C_0603, B.Cu at (32.3, 17.5)
- added C12: 100nF, APRLPrints:C_0603, B.Cu at (146.2, 7.05)
- added C13: 100nF, APRLPrints:C_0603, B.Cu at (152.7, -11.1)
- added C14: 100nF, APRLPrints:C_0603, F.Cu at (257.7, -4.65)
- added C15: ?uF, APRLPrints:C_0603, F.Cu at (254.1, -12.0)
- added C150: 470pF, APRLPrints:C_0603, F.Cu at (112.3, 153.5)
- added C151: 470pF, APRLPrints:C_0603, F.Cu at (111.0, 151.0)
- added C152: 100nF, APRLPrints:C_0603, F.Cu at (111.9, 138.1)
- added C153: 2.2uF, APRLPrints:C_0603, F.Cu at (113.7, 138.1)
- added C154: 100nF, APRLPrints:C_0603, B.Cu at (41.8, -9.16)
- added C155: 100nF, APRLPrints:C_0603, B.Cu at (41.8, -6.71)
- added C156: 100nF, APRLPrints:C_0603, B.Cu at (129.8, -0.02)
- added C157: 10nF, APRLPrints:C_0603, B.Cu at (45.3, -4.26)
- added C158: 100nF, APRLPrints:C_0603, B.Cu at (45.3, -9.16)
- added C159: 10uF, APRLPrints:C_0603, B.Cu at (41.8, -14.1)
- added C16: ?uF, APRLPrints:C_0603, F.Cu at (257.7, -12.0)
- added C160: 10nF, APRLPrints:C_0603, B.Cu at (45.3, -1.81)
- added C161: 100nF, APRLPrints:C_0603, B.Cu at (129.8, -2.47)
- added C162: 100nF, APRLPrints:C_0603, B.Cu at (126.3, -14.7)
- added C163: 100nF, APRLPrints:C_0603, F.Cu at (217.7, -16.7)
- added C164: ?uF, APRLPrints:C_0603, F.Cu at (214.1, -19.1)
- added C165: ?uF, APRLPrints:C_0603, F.Cu at (214.1, -4.45)
- added C166: 100pF, APRLPrints:C_0603, B.Cu at (129.8, 2.43)
- added C167: 100nF, APRLPrints:C_0603, F.Cu at (214.1, -21.6)
- added C168: 100nF, APRLPrints:C_0603, F.Cu at (214.1, -16.7)
- added C169: 100nF, APRLPrints:C_0603, F.Cu at (214.1, -11.8)
- added C17: 100pF, APRLPrints:C_0603, B.Cu at (149.8, -4.05)
- added C170: 100nF, APRLPrints:C_0603, F.Cu at (217.7, -21.6)
- added C171: 100nF, APRLPrints:C_0603, F.Cu at (224.1, -6.00)
- added C172: 30pF, APRLPrints:C_0603, F.Cu at (224.1, -3.55)
- added C173: 22nF, APRLPrints:C_0603, F.Cu at (130.4, 142.2)
- added C174: 22nF, APRLPrints:C_0603, F.Cu at (130.4, 145.1)
- added C175: 100nF, APRLPrints:C_0603, F.Cu at (135.9, 149.7)
- added C176: 100nF, APRLPrints:C_0603, F.Cu at (141.2, 147.8)
- added C177: 100nF, APRLPrints:C_0603, F.Cu at (130.4, 147.8)
- added C178: 100uF, Capacitor_SMD:CP_Elec_10x10.5, F.Cu at (146.1, 140.6)
- added C179: 470pF, APRLPrints:C_0603, F.Cu at (137.4, 153.5)
- added C18: 100nF, APRLPrints:C_0603, F.Cu at (254.1, -14.4)
- added C180: 470pF, APRLPrints:C_0603, F.Cu at (138.8, 151.0)
- added C181: 470pF, APRLPrints:C_0603, F.Cu at (134.4, 153.5)
- added C182: 470pF, APRLPrints:C_0603, F.Cu at (133.0, 151.0)
- added C183: 100nF, APRLPrints:C_0603, F.Cu at (133.7, 138.0)
- added C184: 2.2uF, APRLPrints:C_0603, F.Cu at (135.4, 138.1)
- added C185: 100nF, APRLPrints:C_0603, B.Cu at (205.1, 66.4)
- added C186: 100nF, APRLPrints:C_0603, B.Cu at (117.6, 71.7)
- added C187: 100nF, APRLPrints:C_0603, B.Cu at (214.7, 68.8)
- added C188: 100nF, APRLPrints:C_0603, B.Cu at (214.7, 71.5)
- added C189: 100nF, APRLPrints:C_0603, B.Cu at (204.3, 71.5)
- added C19: 100nF, APRLPrints:C_0603, F.Cu at (254.1, -9.55)
- added C190: 100n, APRLPrints:C_0603, B.Cu at (204.3, 68.7)
- added C191: 100nF, APRLPrints:C_0603, B.Cu at (205.1, 74.0)
- added C192: 100nF, APRLPrints:C_0603, B.Cu at (158.6, 35.6)
- added C193: 100nF, APRLPrints:C_0603, B.Cu at (214.7, 76.2)
- added C194: 100nF, APRLPrints:C_0603, B.Cu at (214.7, 79.0)
- added C195: 100nF, APRLPrints:C_0603, B.Cu at (204.2, 79.0)
- added C196: 100n, APRLPrints:C_0603, B.Cu at (204.2, 76.2)
- added C197: 100nF, APRLPrints:C_0603, B.Cu at (167.6, 147.2)
- added C198: 100nF, APRLPrints:C_0603, B.Cu at (205.1, 81.3)
- added C199: 100nF, APRLPrints:C_0603, B.Cu at (214.7, 83.5)
- added C20: 100nF, APRLPrints:C_0603, F.Cu at (254.1, -4.65)
- added C200: 100nF, APRLPrints:C_0603, B.Cu at (214.7, 86.2)
- added C201: 100nF, APRLPrints:C_0603, B.Cu at (204.4, 86.3)
- added C202: 100n, APRLPrints:C_0603, B.Cu at (204.4, 83.6)
- added C203: 22nF, APRLPrints:C_0603, F.Cu at (152.6, 142.2)
- added C204: 22nF, APRLPrints:C_0603, F.Cu at (152.6, 145.1)
- added C205: 100nF, APRLPrints:C_0603, F.Cu at (158.1, 149.6)
- added C206: 100nF, APRLPrints:C_0603, F.Cu at (163.3, 147.8)
- added C207: 100nF, APRLPrints:C_0603, F.Cu at (152.6, 147.8)
- added C208: 100uF, Capacitor_SMD:CP_Elec_10x10.5, F.Cu at (168.2, 140.6)
- added C209: 470pF, APRLPrints:C_0603, F.Cu at (159.6, 153.5)
- added C210: 470pF, APRLPrints:C_0603, F.Cu at (161.0, 151.0)
- added C211: 470pF, APRLPrints:C_0603, F.Cu at (156.6, 153.5)
- added C212: 470pF, APRLPrints:C_0603, F.Cu at (155.2, 151.0)
- added C213: 100nF, APRLPrints:C_0603, F.Cu at (155.8, 138.0)
- added C214: 2.2uF, APRLPrints:C_0603, F.Cu at (157.6, 138.1)
- added C215: 22nF, APRLPrints:C_0603, F.Cu at (175.1, 142.2)
- added C216: 22nF, APRLPrints:C_0603, F.Cu at (175.1, 145.1)
- added C217: 100nF, APRLPrints:C_0603, F.Cu at (180.6, 149.7)
- added C218: 100nF, APRLPrints:C_0603, F.Cu at (185.8, 147.8)
- added C219: 100nF, APRLPrints:C_0603, F.Cu at (175.1, 147.8)
- added C22: 100nF, APRLPrints:C_0603, F.Cu at (251.1, 8.30)
- added C220: 100uF, Capacitor_SMD:CP_Elec_10x10.5, F.Cu at (190.7, 140.6)
- added C221: 470pF, APRLPrints:C_0603, F.Cu at (182.1, 153.5)
- added C222: 470pF, APRLPrints:C_0603, F.Cu at (183.5, 151.0)
- added C223: 470pF, APRLPrints:C_0603, F.Cu at (179.1, 153.5)
- added C224: 470pF, APRLPrints:C_0603, F.Cu at (177.7, 151.0)
- added C225: 100nF, APRLPrints:C_0603, F.Cu at (178.3, 138.0)
- added C226: 2.2uF, APRLPrints:C_0603, F.Cu at (180.1, 138.1)
- added C227: 22nF, APRLPrints:C_0603, F.Cu at (197.4, 142.2)
- added C228: 22nF, APRLPrints:C_0603, F.Cu at (197.4, 145.1)
- added C229: 100nF, APRLPrints:C_0603, F.Cu at (202.9, 149.7)
- added C230: 100nF, APRLPrints:C_0603, F.Cu at (208.2, 147.8)
- added C231: 100nF, APRLPrints:C_0603, F.Cu at (197.4, 147.8)
- added C232: 100uF, Capacitor_SMD:CP_Elec_10x10.5, F.Cu at (213.1, 140.6)
- added C233: 470pF, APRLPrints:C_0603, F.Cu at (204.5, 153.5)
- added C234: 470pF, APRLPrints:C_0603, F.Cu at (205.9, 151.0)
- added C235: 470pF, APRLPrints:C_0603, F.Cu at (201.4, 153.5)
- added C236: 470pF, APRLPrints:C_0603, F.Cu at (200.1, 151.0)
- added C237: 100nF, APRLPrints:C_0603, F.Cu at (200.7, 138.0)
- added C238: 2.2uF, APRLPrints:C_0603, F.Cu at (202.4, 138.1)
- added C24: 100nF, APRLPrints:C_0603, F.Cu at (202.8, 69.6)
- added C25: 100nF, APRLPrints:C_0603, F.Cu at (212.5, 72.3)
- added C26: 100nF, APRLPrints:C_0603, F.Cu at (213.4, 79.3)
- added C27: 100nF, APRLPrints:C_0603, F.Cu at (215.0, 72.0)
- added C35: 22uF, APRLPrints:C_0805, F.Cu at (121.0, 80.0)
- added C36: 100nF, APRLPrints:C_0603, B.Cu at (78.9, 70.4)
- added C37: 1nF, APRLPrints:C_0603, F.Cu at (120.3, 93.2)
- added C38: 100nF, APRLPrints:C_0603, F.Cu at (111.5, 69.3)
- added C40: 22uF, APRLPrints:C_0805, F.Cu at (106.9, 72.8)
- added C41: 22uF, APRLPrints:C_0805, F.Cu at (109.1, 72.8)
- added C44: 22uF, APRLPrints:C_0805, F.Cu at (122.3, 58.7)
- added C45: 22uF, APRLPrints:C_0805, F.Cu at (124.5, 58.7)
- added C49: 22uF, APRLPrints:C_0805, F.Cu at (135.6, 75.5)
- added C50: 22uF, APRLPrints:C_0805, F.Cu at (135.6, 73.2)
- added C53: 22uF, APRLPrints:C_0805, F.Cu at (139.0, 73.5)
- added C54: 22uF, APRLPrints:C_0805, F.Cu at (138.7, 79.4)
- added C56: 100nF, APRLPrints:C_0603, B.Cu at (106.8, 33.9)
- added C57: 1uF, APRLPrints:C_0603, F.Cu at (154.2, 93.8)
- added C59: 100nF, APRLPrints:C_0603, F.Cu at (154.5, 78.2)
- added C6: 100nF, APRLPrints:C_0603, B.Cu at (28.8, 17.5)
- added C60: 100nF, APRLPrints:C_0603, F.Cu at (183.6, 87.8)
- added C61: 100nF, APRLPrints:C_0603, F.Cu at (166.6, 70.0)
- added C65: 100nF, APRLPrints:C_0603, F.Cu at (172.2, 98.8)
- added C7: 100nF, APRLPrints:C_0603, B.Cu at (160.1, 2.75)
- added C8: 10nF, APRLPrints:C_0603, B.Cu at (35.9, 29.8)
- added C9: 100nF, APRLPrints:C_0603, B.Cu at (35.9, 24.9)
- added D20: LED, APRLPrints:LED_0603, B.Cu at (213.4, 125.9)
- added D21: LED, APRLPrints:LED_0603, B.Cu at (221.9, 126.1)
- added D22: LED_Small, APRLPrints:LED_0603, B.Cu at (123.8, 99.0)
- added D23: ESD9B3.3ST5G, Diode_SMD:D_SOD-923, B.Cu at (126.5, 99.5)
- added D24: LED_Small, APRLPrints:LED_0603, B.Cu at (42.9, 106.5)
- added D25: ESD9B3.3ST5G, Diode_SMD:D_SOD-923, B.Cu at (39.7, 106.2)
- added D26: LED_Small, APRLPrints:LED_0603, B.Cu at (25.4, 106.5)
- added D27: ESD9B3.3ST5G, Diode_SMD:D_SOD-923, B.Cu at (22.2, 106.2)
- added J2: Conn_02x20_Counter_Clockwise, Connector_IDC:IDC-Header_2x20_P2.54mm_Vertical_SMD, F.Cu at (198.0, 125.9)
- added J28: Conn_01x04, libserie:JST_XH_B4B-XH-AM_1x04_P2.50mm_Vertical, F.Cu at (216.2, 30.4)
- added J3: Conn_ARM_SWD_TagConnect_TC2030-NL, Connector:Tag-Connect_TC2030-IDC-NL_2x03_P1.27mm_Vertical, F.Cu at (255.5, 64.6)
- added J35: Conn_01x02, libserie:JST_XH_B2B-XH-AM_1x02_P2.50mm_Vertical, F.Cu at (196.8, 97.3)
- added J36: Conn_01x02, libserie:JST_XH_B2B-XH-AM_1x02_P2.50mm_Vertical, F.Cu at (196.8, 104.3)
- added J37: Conn_01x02, libserie:JST_XH_B2B-XH-AM_1x02_P2.50mm_Vertical, F.Cu at (196.8, 111.3)
- added J38: Conn_01x02, libserie:JST_XH_B2B-XH-AM_1x02_P2.50mm_Vertical, F.Cu at (214.3, 111.4)
- added J39: Conn_01x02, libserie:JST_XH_B2B-XH-AM_1x02_P2.50mm_Vertical, F.Cu at (205.5, 111.4)
- added J4: Conn_01x04, libserie:JST_XH_B4B-XH-AM_1x04_P2.50mm_Vertical, F.Cu at (185.0, 66.2)
- added J40: Conn_01x02, libserie:JST_XH_B2B-XH-AM_1x02_P2.50mm_Vertical, F.Cu at (205.4, 104.4)
- added J41: Conn_01x02, libserie:JST_XH_B2B-XH-AM_1x02_P2.50mm_Vertical, F.Cu at (205.4, 97.4)
- added J42: Conn_01x02, libserie:JST_XH_B2B-XH-AM_1x02_P2.50mm_Vertical, F.Cu at (205.4, 90.4)
- added J43: Conn_01x02, libserie:JST_XH_B2B-XH-AM_1x02_P2.50mm_Vertical, F.Cu at (214.3, 90.4)
- added J44: Conn_01x02, libserie:JST_XH_B2B-XH-AM_1x02_P2.50mm_Vertical, F.Cu at (214.3, 97.4)
- added J45: Conn_01x02, libserie:JST_XH_B2B-XH-AM_1x02_P2.50mm_Vertical, F.Cu at (214.3, 104.4)
- added J46: Conn_01x04, libserie:JST_XH_B4B-XH-AM_1x04_P2.50mm_Vertical, F.Cu at (154.3, 157.8)
- added J47: Conn_01x04, libserie:JST_XH_B4B-XH-AM_1x04_P2.50mm_Vertical, F.Cu at (176.8, 157.8)
- added J48: Conn_01x04, libserie:JST_XH_B4B-XH-AM_1x04_P2.50mm_Vertical, F.Cu at (199.2, 157.8)
- added J49: Conn_01x03, libserie:JST_XH_B3B-XH-AM_1x03_P2.50mm_Vertical, F.Cu at (134.0, 96.3)
- added J5: Conn_01x04, libserie:JST_XH_B4B-XH-AM_1x04_P2.50mm_Vertical, F.Cu at (198.5, 59.0)
- added J50: Conn_01x03, libserie:JST_XH_B3B-XH-AM_1x03_P2.50mm_Vertical, F.Cu at (134.0, 107.3)
- added J51: Conn_01x03, libserie:JST_XH_B3B-XH-AM_1x03_P2.50mm_Vertical, F.Cu at (141.0, 84.8)
- added J6: Conn_01x02, libserie:JST_XH_B2B-XH-AM_1x02_P2.50mm_Vertical, F.Cu at (171.4, 59.0)
- added J7: USB_C_Receptacle_USB2.0_16P, libserie:USB_C_Receptacle_HRO_TYPE-C-31-M-12, F.Cu at (224.5, 82.2)
- added J8: USB_C_Receptacle_USB2.0_16P, libserie:USB_C_Receptacle_HRO_TYPE-C-31-M-12, F.Cu at (224.6, 69.4)
- added J9: Conn_ARM_SWD_TagConnect_TC2030-NL, Connector:Tag-Connect_TC2030-IDC-NL_2x03_P1.27mm_Vertical, F.Cu at (240.6, 59.2)
- added L1: 6.8 uH, Inductor_SMD:L_Changjiang_FXL0630, F.Cu at (120.9, 86.8)
- added L2: 3.3 uH, Inductor_SMD:L_Changjiang_FXL0630, F.Cu at (120.9, 65.4)
- added Q10: AO3400A, Package_TO_SOT_SMD:SOT-23, B.Cu at (55.4, 127.3)
- added Q11: AO3400A, Package_TO_SOT_SMD:SOT-23, B.Cu at (124.3, 96.3)
- added Q12: AO3400A, Package_TO_SOT_SMD:SOT-23, B.Cu at (47.2, 107.5)
- added Q13: AO3400A, Package_TO_SOT_SMD:SOT-23, B.Cu at (29.7, 107.5)
- added Q8: AO3400A, Package_TO_SOT_SMD:SOT-23, B.Cu at (29.7, 121.7)
- added Q9: AO3400A, Package_TO_SOT_SMD:SOT-23, B.Cu at (41.1, 50.8)
- added R1: 100R, APRLPrints:R_0603, B.Cu at (28.8, 22.4)
- added R10: 4.7k, APRLPrints:R_0603, B.Cu at (152.1, -3.45)
- added R100: 10k, APRLPrints:R_0603, B.Cu at (215.5, 66.6)
- added R101: 10k, APRLPrints:R_0603, B.Cu at (259.1, 73.0)
- added R102: 10k, APRLPrints:R_0603, B.Cu at (258.5, 74.8)
- added R103: 4.7k, APRLPrints:R_0603, B.Cu at (216.2, 76.2)
- added R104: 4.7k, APRLPrints:R_0603, B.Cu at (216.2, 79.0)
- added R105: 4.7k, APRLPrints:R_0603, B.Cu at (205.8, 79.0)
- added R106: 4.7k, APRLPrints:R_0603, B.Cu at (205.8, 76.2)
- added R107: 10k, APRLPrints:R_0603, B.Cu at (215.4, 74.0)
- added R108: 4.7k, APRLPrints:R_0603, B.Cu at (216.3, 83.5)
- added R109: 4.7k, APRLPrints:R_0603, B.Cu at (216.3, 86.2)
- added R11: 100k, APRLPrints:R_0603, B.Cu at (152.1, -5.25)
- added R110: 4.7k, APRLPrints:R_0603, B.Cu at (206.0, 86.3)
- added R111: 4.7k, APRLPrints:R_0603, B.Cu at (206.0, 83.6)
- added R112: 10k, APRLPrints:R_0603, B.Cu at (215.5, 81.3)
- added R113: 24k, APRLPrints:R_0603, F.Cu at (159.3, 138.1)
- added R114: 24k, APRLPrints:R_0603, F.Cu at (181.8, 138.1)
- added R115: 24k, APRLPrints:R_0603, F.Cu at (204.2, 138.1)
- added R116: 10k, APRLPrints:R_0603, B.Cu at (128.6, 99.0)
- added R117: 10k, APRLPrints:R_0603, B.Cu at (123.7, 100.9)
- added R118: 4.7k, APRLPrints:R_0603, B.Cu at (128.6, 100.6)
- added R119: 10R, APRLPrints:R_0603, B.Cu at (129.0, 96.3)
- added R12: 10M, APRLPrints:R_0603, B.Cu at (148.2, -4.05)
- added R120: 100k, APRLPrints:R_0603, B.Cu at (127.3, 96.3)
- added R121: 10k, APRLPrints:R_0603, B.Cu at (51.5, 106.0)
- added R122: 10k, APRLPrints:R_0603, B.Cu at (51.5, 101.1)
- added R123: 4.7k, APRLPrints:R_0603, B.Cu at (51.5, 108.5)
- added R124: 10R, APRLPrints:R_0603, B.Cu at (51.5, 98.7)
- added R125: 100k, APRLPrints:R_0603, B.Cu at (51.5, 103.5)
- added R126: 10k, APRLPrints:R_0603, B.Cu at (34.0, 106.0)
- added R127: 10k, APRLPrints:R_0603, B.Cu at (34.0, 101.1)
- added R128: 4.7k, APRLPrints:R_0603, B.Cu at (34.0, 108.5)
- added R129: 10R, APRLPrints:R_0603, B.Cu at (34.0, 98.7)
- added R13: 10k, APRLPrints:R_0603, B.Cu at (147.8, 7.05)
- added R130: 100k, APRLPrints:R_0603, B.Cu at (34.0, 103.5)
- added R14: 10k, APRLPrints:R_0603, B.Cu at (150.2, 7.65)
- added R15: 10k, APRLPrints:R_0603, F.Cu at (223.0, 91.5)
- added R16: 4.7k, APRLPrints:R_0603, F.Cu at (218.0, 79.7)
- added R17: 4.7k, APRLPrints:R_0603, F.Cu at (218.0, 84.8)
- added R18: 10k, APRLPrints:R_0603, F.Cu at (200.6, 71.7)
- added R19: 10k, APRLPrints:R_0603, F.Cu at (200.6, 73.3)
- added R2: 100R, APRLPrints:R_0603, B.Cu at (28.8, 19.9)
- added R20: 10k, APRLPrints:R_0603, F.Cu at (200.6, 74.9)
- added R21: 4.7k, APRLPrints:R_0603, F.Cu at (218.0, 67.0)
- added R3: 4.7k, APRLPrints:R_0603, B.Cu at (157.2, 8.40)
- added R30: 200k, APRLPrints:R_0603, F.Cu at (112.7, 76.4)
- added R31: 10k, APRLPrints:R_0603, F.Cu at (116.1, 76.4)
- added R32: 30.9k, APRLPrints:R_0603, F.Cu at (120.3, 73.8)
- added R33: 10k, APRLPrints:R_0603, F.Cu at (133.8, 66.5)
- added R35: 10R, APRLPrints:R_0603, F.Cu at (103.5, 98.0)
- added R36: 100k, APRLPrints:R_0603, F.Cu at (103.5, 95.2)
- added R37: 10k, APRLPrints:R_0603, F.Cu at (95.6, 113.9)
- added R38: 10R, APRLPrints:R_0603, F.Cu at (98.8, 102.0)
- added R4: 4.7k, APRLPrints:R_0603, F.Cu at (155.9, 4.17)
- added R5: 4.7k, APRLPrints:R_0603, B.Cu at (154.4, 8.40)
- added R6: 4.7k, APRLPrints:R_0603, F.Cu at (154.3, 2.35)
- added R7: 4.7k, APRLPrints:R_0603, B.Cu at (157.8, -2.40)
- added R8: 4.7k, APRLPrints:R_0603, B.Cu at (155.0, -2.40)
- added R82: 100R, APRLPrints:R_0603, B.Cu at (38.2, -14.1)
- added R83: 4.7k, APRLPrints:R_0603, B.Cu at (126.3, 2.43)
- added R84: 4.7k, APRLPrints:R_0603, B.Cu at (122.8, -14.7)
- added R85: 4.7k, APRLPrints:R_0603, B.Cu at (122.8, -12.3)
- added R86: 4.7k, APRLPrints:R_0603, B.Cu at (122.8, -9.82)
- added R87: 4.7k, APRLPrints:R_0603, B.Cu at (122.8, -7.37)
- added R88: 4.7k, APRLPrints:R_0603, B.Cu at (122.8, -4.92)
- added R89: 4.7k, APRLPrints:R_0603, B.Cu at (122.8, -2.47)
- added R9: 4.7k, APRLPrints:R_0603, B.Cu at (152.7, -0.65)
- added R90: 4.7k, APRLPrints:R_0603, B.Cu at (122.8, -0.02)
- added R91: 100k, APRLPrints:R_0603, B.Cu at (126.3, -4.92)
- added R92: 10M, APRLPrints:R_0603, B.Cu at (126.3, -7.37)
- added R93: 10k, APRLPrints:R_0603, B.Cu at (126.3, -2.47)
- added R94: 10k, APRLPrints:R_0603, B.Cu at (126.3, -0.02)
- added R95: 24k, APRLPrints:R_0603, F.Cu at (137.2, 138.1)
- added R96: 4.7k, APRLPrints:R_0603, B.Cu at (216.3, 68.8)
- added R97: 4.7k, APRLPrints:R_0603, B.Cu at (216.3, 71.5)
- added R98: 4.7k, APRLPrints:R_0603, B.Cu at (205.9, 71.5)
- added R99: 4.7k, APRLPrints:R_0603, B.Cu at (205.9, 68.7)
- added REF**: Loose Pads, APRLPrints:Loose Pads, F.Cu at (191.5, 153.0)
- added REF**: Loose Pads, APRLPrints:Loose Pads, F.Cu at (125.2, 153.0)
- added REF**: Loose Pads, APRLPrints:Loose Pads, F.Cu at (99.2, 87.0)
- added REF**: Loose Pads, APRLPrints:Loose Pads, F.Cu at (146.4, 153.2)
- added U10: USBLC6-2SC6, Package_TO_SOT_SMD:SOT-23-6, F.Cu at (214.3, 69.3)
- added U2: ADS1220xPW, Package_SO:TSSOP-16_4.4x5mm_P0.65mm, B.Cu at (42.3, 35.2)
- added U3: TMUX1108PW, Package_SO:TSSOP-16_4.4x5mm_P0.65mm, B.Cu at (156.4, 3.20)
- added U30: ADS1220xPW, Package_SO:TSSOP-16_4.4x5mm_P0.65mm, B.Cu at (18.7, -14.4)
- added U31: TMUX1108PW, Package_SO:TSSOP-16_4.4x5mm_P0.65mm, B.Cu at (106.8, -6.06)
- added U32: TLV6742, Package_SO:SOIC-8_3.9x4.9mm_P1.27mm, B.Cu at (107.3, 0.59)
- added U33: TLV6742, Package_SO:SOIC-8_3.9x4.9mm_P1.27mm, B.Cu at (107.3, 7.18)
- added U34: LDC1612, libserie:WSON-12-1EP_4x4mm_P0.5mm_EP2.6x3mm_ThermalVias, F.Cu at (231.5, -12.2)
- added U35: TMUX1101DBV, Package_TO_SOT_SMD:SOT-23-5, B.Cu at (126.6, 5.60)
- added U36: TMC2241ATC, libserie:QFN-38_EP_5.63x7.6_Pitch0.5mm, F.Cu at (135.9, 143.7)
- added U37: ADS1115IDGS, Package_SO:TSSOP-10_3x3mm_P0.5mm, B.Cu at (210.4, 69.0)
- added U38: LM75B, Package_SO:SOIC-8_3.9x4.9mm_P1.27mm, B.Cu at (118.8, 67.0)
- added U39: ADS1115IDGS, Package_SO:TSSOP-10_3x3mm_P0.5mm, B.Cu at (210.4, 76.6)
- added U40: LM75B, Package_SO:SOIC-8_3.9x4.9mm_P1.27mm, B.Cu at (157.4, 40.4)
- added U41: LM75B, Package_SO:SOIC-8_3.9x4.9mm_P1.27mm, B.Cu at (168.8, 142.6)
- added U42: ADS1115IDGS, Package_SO:TSSOP-10_3x3mm_P0.5mm, B.Cu at (210.4, 84.3)
- added U43: TMC2241ATC, libserie:QFN-38_EP_5.63x7.6_Pitch0.5mm, F.Cu at (158.1, 143.7)
- added U44: TMC2241ATC, libserie:QFN-38_EP_5.63x7.6_Pitch0.5mm, F.Cu at (180.6, 143.7)
- added U45: TMC2241ATC, libserie:QFN-38_EP_5.63x7.6_Pitch0.5mm, F.Cu at (202.9, 143.7)
- added U7: TMUX1101DBV, Package_TO_SOT_SMD:SOT-23-5, B.Cu at (143.9, -3.50)
- added Y2: 12 MHz, APRLPrints:3225-4P-L, F.Cu at (257.1, 2.90)
- added Y3: 12 MHz, APRLPrints:3225-4P-L, F.Cu at (217.1, 0.65)
- C1, C2: value 2.2uF -> 10pF
- C100, C112, C124, C136, C148, C88: value 100uF -> 470pF; footprint Capacitor_SMD:CP_Elec_10x10.5 -> APRLPrints:C_0603
- C102, C114, C126, C138, C90: value 100nF -> 470pF
- C103, C115, C127, C139, C91: value 2.2uF -> 470pF
- C104, C116, C128, C140, C92: value 22nF -> 100nF
- C105, C117, C129, C141, C93: value 22nF -> 2.2uF
- C106, C118, C130, C142, C82, C94: value 100nF -> 22nF
- C107, C119, C131, C143, C83, C95: value 470pF -> 22nF
- C109, C121, C133, C145, C85, C97: value 470pF -> 100nF
- C110, C122, C134, C146, C86, C98: value 100uF -> 100nF; footprint Capacitor_SMD:CP_Elec_10x10.5 -> APRLPrints:C_0603
- C111, C123, C135, C147, C87, C99: value 470pF -> 100uF; footprint APRLPrints:C_0603 -> Capacitor_SMD:CP_Elec_10x10.5
- C23: value 100nF -> 30pF
- C29, C30, C31, C48, C51, C52, C55: value 100nF -> 22uF; footprint APRLPrints:C_0603 -> APRLPrints:C_0805
- C3: value 100nF -> 2.2uF; moved to B.Cu
- C32, C42: value 22uF -> 100uF; footprint APRLPrints:C_0805 -> Capacitor_SMD:CP_Elec_10x10.5
- C4: value 10pF -> 2.2uF; moved to B.Cu
- C47: value 100nF -> 1nF
- C5: value 10pF -> 100nF; moved to B.Cu
- C69, C71: value 1uF -> 100nF
- C72: value 10nF -> 100nF
- C73: value 100nF -> 1uF
- C75: value 10nF -> 1uF
- C76, C77, D14, D16, R46, R50, R51, R52, R55, R57, R59, R62, R63, R64, R65, R66, R67, R68, R69, R72, U20, U21: moved to B.Cu
- C78: value 100nF -> 10nF; moved to B.Cu
- C79: value 2.2uF -> 100nF; moved to B.Cu
- C80: value 22nF -> 100nF; moved to B.Cu
- C81: value 22nF -> 10nF; moved to B.Cu
- D1: value LED_Small -> PMEG3010BER; footprint APRLPrints:LED_0603 -> Diode_SMD:Nexperia_CFP3_SOD-123W
- D15, D17: value LED_Small -> ESD9B3.3ST5G; footprint APRLPrints:LED_0603 -> Diode_SMD:D_SOD-923; moved to B.Cu
- D18: value LED -> LED_Small; moved to B.Cu
- D19: value LED -> ESD9B3.3ST5G; footprint APRLPrints:LED_0603 -> Diode_SMD:D_SOD-923; moved to B.Cu
- D2: value PMEG3010BER -> LED_Small; footprint Diode_SMD:Nexperia_CFP3_SOD-123W -> APRLPrints:LED_0603
- D6, D8: value SS54 -> LED_Small; footprint Diode_SMD:D_SMA -> APRLPrints:LED_0603
- D7: value LED_Small -> SS54; footprint APRLPrints:LED_0603 -> Diode_SMD:D_SMA
- F2: value XFCN XF-508P-B-B -> XF-508P-B-B
- J1: value Conn_02x05_Odd_Even -> Conn_02x20_Counter_Clockwise; footprint Connector_PinHeader_2.54mm:PinHeader_1x10_P2.54mm_Vertical -> Connector_IDC:IDC-Header_2x20_P2.54mm_Vertical_SMD
- J10: value Screw_Terminal_01x02 -> Screw_Terminal_06x01x02; footprint Connector_Phoenix_MSTB:PhoenixContact_MSTBA_2,5_2-G_1x02_P5.00mm_Horizontal -> TerminalBlock_Ningbo-Kagnex:TerminalBlock_Ningbo-Kagnex_HB9500M_1x12_P9.5mm
- J11, J12: value USB_C_Receptacle_USB2.0_16P -> Conn_01x03; footprint Connector_USB:USB_C_Receptacle_HRO_TYPE-C-31-M-12 -> libserie:JST_XH_B3B-XH-AM_1x03_P2.50mm_Vertical
- J13: value Conn_02x05_Odd_Even -> Conn_01x03; footprint Connector_PinHeader_2.54mm:PinHeader_2x05_P2.54mm_Vertical -> libserie:JST_XH_B3B-XH-AM_1x03_P2.50mm_Vertical
- J14: value Screw_Terminal_06x01x02 -> Conn_01x03; footprint TerminalBlock_Ningbo-Kagnex:TerminalBlock_Ningbo-Kagnex_HB9500M_1x12_P9.5mm -> libserie:JST_XH_B3B-XH-AM_1x03_P2.50mm_Vertical
- J15, J16, J17, J18: value Conn_01x02 -> Conn_01x03; footprint Connector_Molex:Molex_Micro-Fit_3.0_43650-0215_1x02_P3.00mm_Vertical -> libserie:JST_XH_B3B-XH-AM_1x03_P2.50mm_Vertical
- J19, J20, J21: footprint Connector_Molex:Molex_Micro-Fit_3.0_43650-0315_1x03_P3.00mm_Vertical -> libserie:JST_XH_B3B-XH-AM_1x03_P2.50mm_Vertical
- J22, J23: value Conn_01x03 -> Conn_01x02; footprint Connector_Molex:Molex_Micro-Fit_3.0_43650-0315_1x03_P3.00mm_Vertical -> libserie:JST_XH_B2B-XH-AM_1x02_P2.50mm_Vertical
- J24, J25, J26: value Conn_01x03 -> Conn_01x04; footprint Connector_Molex:Molex_Micro-Fit_3.0_43650-0315_1x03_P3.00mm_Vertical -> libserie:JST_XH_B4B-XH-AM_1x04_P2.50mm_Vertical
- J27: value Conn_01x02 -> Conn_01x04; footprint Connector_Molex:Molex_Micro-Fit_3.0_43650-0215_1x02_P3.00mm_Vertical -> libserie:JST_XH_B4B-XH-AM_1x04_P2.50mm_Vertical
- J29, J30, J31, J33: footprint Connector_JST:JST_XH_B4B-XH-AM_1x04_P2.50mm_Vertical -> libserie:JST_XH_B4B-XH-AM_1x04_P2.50mm_Vertical
- J32, J34: value Conn_01x04 -> Conn_01x02; footprint Connector_JST:JST_XH_B4B-XH-AM_1x04_P2.50mm_Vertical -> libserie:JST_XH_B2B-XH-AM_1x02_P2.50mm_Vertical
- Q1, Q3: value CSD18532NQ5B -> BSC016N06NS; moved to B.Cu
- Q2, Q4: value CSD18532NQ5B -> BSC016N06NS
- Q5, Q6, Q7: value AO3400A -> BSC016N06NS; footprint Package_TO_SOT_SMD:SOT-23 -> Package_TO_SOT_SMD:TDSON-8-1
- R23, R25: value 4.7k -> 10k
- R24: value 4.7k -> 140k
- R26: value 10k -> 200k
- R27: value 10k -> 30.9k
- R29: value 10k -> 52.5k
- R39, R45: value 10k -> 100k
- R42: value 10R -> 100k
- R43: value 100k -> 10k
- R44: value 100k -> 10R
- R47, R56: value 10R -> 10k; moved to B.Cu
- R48, R53: value 10R -> 4.7k; moved to B.Cu
- R49: value 100k -> 10R; moved to B.Cu
- R54: value 10k -> 10R; moved to B.Cu
- R58: value 100k -> 4.7k; moved to B.Cu
- R60: value 10k -> 100k; moved to B.Cu
- R61: value 100k -> 10k; moved to B.Cu
- R70, R73: value 4.02k -> 10k; moved to B.Cu
- R71, R74: value 10k -> 4.02k; moved to B.Cu
- R75: value 10k -> 24k
- R81: value 24k -> 100R; moved to B.Cu
- U11: value USBLC6-2SC6 -> AP64500; footprint Package_TO_SOT_SMD:SOT-23-6 -> libserie:Diodes_SO-8EP
- U12: value USBLC6-2SC6 -> AP74700Q; footprint Package_TO_SOT_SMD:SOT-23-6 -> libserie:SOT-6; moved to B.Cu
- U13: value STM32F042F4Px -> AP64500; footprint Package_SO:TSSOP-20_4.4x6.5mm_P0.65mm -> libserie:Diodes_SO-8EP
- U14: value AP2112K-3.3 -> AP74700Q; footprint Package_TO_SOT_SMD:SOT-23-5 -> libserie:SOT-6
- U15: value AP64500 -> TLV77533; footprint Package_SO:Diodes_SO-8EP -> Package_TO_SOT_SMD:SOT-23-5
- U16: value AP64500 -> TPS7A20xxxDQN; footprint Package_SO:Diodes_SO-8EP -> Package_SON:Texas_X2SON-4_1x1mm_P0.65mm
- U17: value TPS7A20xxxDQN -> AP74700Q; footprint Package_SON:Texas_X2SON-4_1x1mm_P0.65mm -> libserie:SOT-6; moved to B.Cu
- U18, U19: footprint Package_SO:Texas_DGN0008G_VSSOP-8-1EP_3x3mm_P0.65mm_EP2x2.94mm_Mask1.846x2.15mm_ThermalVias -> libserie:Texas_DGN0008G_VSSOP-8-1EP_3x3mm_P0.65mm_EP2x2.94mm_Mask1.846x2.15mm_ThermalVias
- U22, U23: footprint Package_DFN_QFN:TQFN-20-1EP_5x5mm_P0.65mm_EP3.25x3.25mm -> libserie:TQFN-20-1EP_5x5mm_P0.65mm_EP3.25x3.25mm; moved to B.Cu
- U4: value LDC1612 -> TLV6742; footprint Package_SON:WSON-12-1EP_4x4mm_P0.5mm_EP2.6x3mm_ThermalVias -> Package_SO:SOIC-8_3.9x4.9mm_P1.27mm; moved to B.Cu
- U5: value ADS1115IDGS -> TLV6742; footprint Package_SO:TSSOP-10_3x3mm_P0.5mm -> Package_SO:SOIC-8_3.9x4.9mm_P1.27mm; moved to B.Cu
- U6: value ADS1220xPW -> LDC1612; footprint Package_SO:TSSOP-16_4.4x5mm_P0.65mm -> libserie:WSON-12-1EP_4x4mm_P0.5mm_EP2.6x3mm_ThermalVias
- U8: value TMUX1101DBV -> USBLC6-2SC6; footprint Package_TO_SOT_SMD:SOT-23-5 -> Package_TO_SOT_SMD:SOT-23-6
- U9: value TMUX1108PW -> STM32F042F4Px; footprint Package_SO:TSSOP-16_4.4x5mm_P0.65mm -> Package_SO:TSSOP-20_4.4x6.5mm_P0.65mm
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Connections:
- net /Connections/OUT3 renamed /Connections/Low Power Outputs/OUT_LP_3
- net /Connections/Sensors/SCLK renamed /Connections/Sensors 1/SCL
- net /Connections/Sensors/~{LC_CS} renamed /Connections/Sensors 1/SDA
- C1 pad 2: Net-(C1-Pad2) -> Net-(U1H-PH1)
- C100 pad 1: VM -> Net-(J25-Pin_3)
- C101 pad 1: Net-(J30-Pin_2) -> Net-(J25-Pin_4)
- C102 pad 1: GND -> Net-(J25-Pin_2)
- C102 pad 2: +3.3V -> GND
- C103 pad 1: GND -> Net-(J25-Pin_1)
- C103 pad 2: Net-(U26-VDD18) -> GND
- C104 pad 1: Net-(U26-CPO) -> GND
- C104 pad 2: Net-(U26-CPI) -> +3.3V
- C105 pad 1: VM -> GND
- C105 pad 2: Net-(U26-VCP) -> Net-(U25-VDD18)
- C106 pad 1: VM -> Net-(U26-CPO)
- C106 pad 2: GND -> Net-(U26-CPI)
- C107 pad 1: Net-(J31-Pin_4) -> VM
- C107 pad 2: GND -> Net-(U26-VCP)
- C109 pad 1: Net-(J31-Pin_3) -> VM
- C111 pad 1: Net-(J31-Pin_1) -> VM
- C112 pad 1: VM -> Net-(J26-Pin_3)
- C113 pad 1: Net-(J31-Pin_2) -> Net-(J26-Pin_4)
- C114 pad 1: GND -> Net-(J26-Pin_2)
- C114 pad 2: +3.3V -> GND
- C115 pad 1: GND -> Net-(J26-Pin_1)
- C115 pad 2: Net-(U27-VDD18) -> GND
- C116 pad 1: Net-(U27-CPO) -> GND
- C116 pad 2: Net-(U27-CPI) -> +3.3V
- C117 pad 1: VM -> GND
- C117 pad 2: Net-(U27-VCP) -> Net-(U26-VDD18)
- C118 pad 1: VM -> Net-(U27-CPO)
- C118 pad 2: GND -> Net-(U27-CPI)
- C119 pad 1: Net-(J32-Pin_4) -> VM
- C119 pad 2: GND -> Net-(U27-VCP)
- C121 pad 1: Net-(J32-Pin_3) -> VM
- C123 pad 1: Net-(J32-Pin_1) -> VM
- C124 pad 1: VM -> Net-(J27-Pin_3)
- C125 pad 1: Net-(J32-Pin_2) -> Net-(J27-Pin_4)
- C126 pad 1: GND -> Net-(J27-Pin_2)
- C126 pad 2: +3.3V -> GND
- C127 pad 1: GND -> Net-(J27-Pin_1)
- C127 pad 2: Net-(U28-VDD18) -> GND
- C128 pad 1: Net-(U28-CPO) -> GND
- C128 pad 2: Net-(U28-CPI) -> +3.3V
- C129 pad 1: VM -> GND
- C129 pad 2: Net-(U28-VCP) -> Net-(U27-VDD18)
- C130 pad 1: VM -> Net-(U28-CPO)
- C130 pad 2: GND -> Net-(U28-CPI)
- C131 pad 1: Net-(J33-Pin_4) -> VM
- C131 pad 2: GND -> Net-(U28-VCP)
- C133 pad 1: Net-(J33-Pin_3) -> VM
- C135 pad 1: Net-(J33-Pin_1) -> VM
- C136 pad 1: VM -> Net-(J28-Pin_3)
- C137 pad 1: Net-(J33-Pin_2) -> Net-(J28-Pin_4)
- C138 pad 1: GND -> Net-(J28-Pin_2)
- C138 pad 2: +3.3V -> GND
- C139 pad 1: GND -> Net-(J28-Pin_1)
- C139 pad 2: Net-(U29-VDD18) -> GND
- C140 pad 1: Net-(U29-CPO) -> GND
- C140 pad 2: Net-(U29-CPI) -> +3.3V
- C141 pad 1: VM -> GND
- C141 pad 2: Net-(U29-VCP) -> Net-(U28-VDD18)
- C142 pad 1: VM -> Net-(U29-CPO)
- C142 pad 2: GND -> Net-(U29-CPI)
- C143 pad 1: Net-(J34-Pin_4) -> VM
- C143 pad 2: GND -> Net-(U29-VCP)
- C145 pad 1: Net-(J34-Pin_3) -> VM
- C147 pad 1: Net-(J34-Pin_1) -> VM
- C148 pad 1: VM -> Net-(J29-Pin_3)
- C149 pad 1: Net-(J34-Pin_2) -> Net-(J29-Pin_4)
- C2 pad 2: Net-(C2-Pad2) -> Net-(U1H-PH0)
- C21 pad 2: +3.3V -> Net-(J5-Pin_1)
- C23 pad 1: +4.5V -> /Connections/Sensors 1/CLK
- C28 pad 1: Net-(U11-VBUS) -> Net-(U11-SW)
- C28 pad 2: GND -> Net-(U11-BST)
- C29 pad 1: Net-(U12-VBUS) -> +24V
- C3 pad 2: +3.3V -> Net-(C3-Pad2)
- C30 pad 1: +3.3V -> +24V
- C31 pad 1: +3.3V -> +24V
- C32 pad 1: GND -> +12V
- C32 pad 2: +5V -> GND
- C33 pad 1: GND -> +12V
- C33 pad 2: +5V -> GND
- C34 pad 1: GND -> +12V
- C34 pad 2: +5V -> GND
- C39 pad 1: GND -> +24V
- C39 pad 2: +3.3V -> GND
- C4 pad 2: Net-(U1H-PH1) -> Net-(C4-Pad2)
- C42 pad 1: GND -> Net-(D7-A)
- C42 pad 2: +3.3V -> GND
- C43 pad 1: GND -> Net-(D7-A)
- C43 pad 2: +3.3V -> GND
- C46 pad 1: GND -> Net-(U14-VCP)
- C46 pad 2: +3.3V -> Net-(D7-K)
- C47 pad 1: GND -> Net-(C47-Pad1)
- C47 pad 2: +3.3V -> GND
- C48 pad 2: +3.3V -> +5V
- C5 pad 2: Net-(U1H-PH0) -> +3.3V
- C55 pad 1: GND -> +4.5V
- C55 pad 2: +3.3V -> GND
- C68 pad 2: +12V -> +3.3V
- C69 pad 2: +12V -> +3.3V
- C70 pad 2: +12V -> +3.3V
- C71 pad 2: +12V -> +3.3V
- C72 pad 1: /Connections/Thermocouple 1/T1+ -> GND
- C72 pad 2: /Connections/Thermocouple 1/T1- -> +12V
- C73 pad 1: +3V3 -> GND
- C73 pad 2: GND -> +12V
- C74 pad 1: +3V3 -> GND
- C74 pad 2: GND -> +12V
- C75 pad 1: /Connections/Thermocouple 2/T1+ -> GND
- C75 pad 2: /Connections/Thermocouple 2/T1- -> +12V
- C76 pad 1: +3V3 -> +3.3V
- C77 pad 1: +3V3 -> +3.3V
- C78 pad 1: GND -> /Connections/Thermocouple 1/T1+
- C78 pad 2: +3.3V -> /Connections/Thermocouple 1/T1-
- C79 pad 1: GND -> +3.3V
- C79 pad 2: Net-(U24-VDD18) -> GND
- C80 pad 1: Net-(U24-CPO) -> +3.3V
- C80 pad 2: Net-(U24-CPI) -> GND
- C81 pad 1: VM -> /Connections/Thermocouple 2/T1+
- C81 pad 2: Net-(U24-VCP) -> /Connections/Thermocouple 2/T1-
- C82 pad 1: VM -> Net-(U24-CPO)
- C82 pad 2: GND -> Net-(U24-CPI)
- C83 pad 1: Net-(J29-Pin_4) -> VM
- C83 pad 2: GND -> Net-(U24-VCP)
- C85 pad 1: Net-(J29-Pin_3) -> VM
- C87 pad 1: Net-(J29-Pin_1) -> VM
- C88 pad 1: VM -> Net-(J24-Pin_3)
- C89 pad 1: Net-(J29-Pin_2) -> Net-(J24-Pin_4)
- C90 pad 1: GND -> Net-(J24-Pin_2)
- C90 pad 2: +3.3V -> GND
- C91 pad 1: GND -> Net-(J24-Pin_1)
- C91 pad 2: Net-(U25-VDD18) -> GND
- C92 pad 1: Net-(U25-CPO) -> GND
- C92 pad 2: Net-(U25-CPI) -> +3.3V
- C93 pad 1: VM -> GND
- C93 pad 2: Net-(U25-VCP) -> Net-(U24-VDD18)
- C94 pad 1: VM -> Net-(U25-CPO)
- C94 pad 2: GND -> Net-(U25-CPI)
- C95 pad 1: Net-(J30-Pin_4) -> VM
- C95 pad 2: GND -> Net-(U25-VCP)
- C97 pad 1: Net-(J30-Pin_3) -> VM
- C99 pad 1: Net-(J30-Pin_1) -> VM
- D1 pad 1: GND -> +5V
- D10 pad 1: GND -> Net-(D10-K)
- D15 pad 1: Net-(D15-K) -> GND
- D15 pad 2: Net-(D15-A) -> /Connections/Low Power Outputs/TACH1
- D17 pad 1: Net-(D17-K) -> GND
- D17 pad 2: Net-(D17-A) -> /Connections/Low Power Outputs/TACH2
- D18 pad 1: /Connections/~{DRV_DRDY_1} -> Net-(D18-K)
- D19 pad 1: /Connections/~{DRV_DRDY_2} -> GND
- D19 pad 2: Net-(D19-A) -> /Connections/Low Power Outputs/TACH3
- D2 pad 1: +5V -> GND
- D6 pad 1: +24V -> GND
- D6 pad 2: GND -> Net-(D6-A)
- D7 pad 1: GND -> Net-(D7-K)
- D8 pad 1: +VM -> GND
- D8 pad 2: GND -> Net-(D8-A)
- F1 pad 1: Net-(U11-VBUS) -> Net-(U8-VBUS)
- F1 pad 2: Net-(D2-A) -> Net-(D1-A)
- F2 pad 1: +24V -> Net-(F2-Pad1)
- F2 pad 2: Net-(J14A-Pin_2) -> Net-(J10B-Pin_2)
- F3 pad 1: +VM -> Net-(U17-ANODE)
- F3 pad 2: Net-(J14B-Pin_2) -> Net-(J10A-Pin_2)
- J1 pad 1: +3.3V -> GND
- J1 pad 10: /Connections/~{RST} -> unconnected-(J1-Pin_10-Pad10)
- J1 pad 2: /Connections/SWDIO -> unconnected-(J1-Pin_2-Pad2)
- J1 pad 4: /Connections/SWCLK -> unconnected-(J1-Pin_4-Pad4)
- J1 pad 6: /Connections/SWO -> unconnected-(J1-Pin_6-Pad6)
- J1 pad 7: unconnected-(J1-Pin_7-Pad7) -> GND
- J10 pad 2: Net-(J10-Pin_2) -> Net-(J10A-Pin_2)
- J13 pad 1: +3.3V -> +12V
- J13 pad 2: /Connections/Debugger and USB/IF_SWDIO -> Net-(D18-K)
- J13 pad 3: GND -> Net-(J13-Pin_3)
- J14 pad 2: Net-(J14A-Pin_2) -> Net-(J14-Pin_2)
- J14 pad 3: GND -> +3.3V
- J15 pad 1: /Connections/Thermocouple 2/T1- -> GND
- J15 pad 2: /Connections/Thermocouple 2/T1+ -> Net-(J15-Pin_2)
- J16 pad 1: +12V -> GND
- J16 pad 2: Net-(D15-K) -> Net-(J16-Pin_2)
- J17 pad 1: +12V -> GND
- J17 pad 2: Net-(D16-K) -> Net-(J17-Pin_2)
- J18 pad 1: +12V -> GND
- J18 pad 2: Net-(D17-K) -> Net-(J18-Pin_2)
- J22 pad 1: GND -> /Connections/Thermocouple 1/T1-
- J22 pad 2: Net-(J22-Pin_2) -> /Connections/Thermocouple 1/T1+
- J23 pad 1: GND -> /Connections/Thermocouple 2/T1-
- J23 pad 2: Net-(J23-Pin_2) -> /Connections/Thermocouple 2/T1+
- J24 pad 1: GND -> Net-(J24-Pin_1)
- J24 pad 3: +3.3V -> Net-(J24-Pin_3)
- J25 pad 1: GND -> Net-(J25-Pin_1)
- J25 pad 3: +3.3V -> Net-(J25-Pin_3)
- J26 pad 1: GND -> Net-(J26-Pin_1)
- J26 pad 3: +3.3V -> Net-(J26-Pin_3)
- J27 pad 1: /Connections/Thermocouple 1/T1- -> Net-(J27-Pin_1)
- J27 pad 2: /Connections/Thermocouple 1/T1+ -> Net-(J27-Pin_2)
- J30 pad 4: Net-(J30-Pin_4) -> +4.5V
- J32 pad 1: Net-(J32-Pin_1) -> GND
- J34 pad 1: Net-(J34-Pin_1) -> GND
- Q1 pad 1: GND -> Net-(F2-Pad1)
- Q1 pad 2: GND -> Net-(F2-Pad1)
- Q1 pad 3: GND -> Net-(F2-Pad1)
- Q1 pad 5: Net-(D11-K) -> +24V
- Q2 pad 1: GND -> Net-(D7-K)
- Q2 pad 2: GND -> Net-(D7-K)
- Q2 pad 3: GND -> Net-(D7-K)
- Q2 pad 5: Net-(D12-K) -> +5V
- Q3 pad 1: GND -> Net-(U17-ANODE)
- Q3 pad 2: GND -> Net-(U17-ANODE)
- Q3 pad 3: GND -> Net-(U17-ANODE)
- Q3 pad 5: Net-(D13-K) -> VM
- Q4 pad 5: Net-(D14-K) -> Net-(D10-K)
- Q5 pad 1: Net-(Q5-G) -> GND
- Q5 pad 3: Net-(D15-K) -> GND
- Q6 pad 1: Net-(Q6-G) -> GND
- Q6 pad 3: Net-(D16-K) -> GND
- Q7 pad 1: Net-(Q7-G) -> GND
- Q7 pad 3: Net-(D17-K) -> GND
- R22 pad 1: GND -> Net-(J8-CC1)
- R22 pad 2: Net-(J11-CC2) -> GND
- R23 pad 1: GND -> +12V
- R23 pad 2: Net-(J12-CC2) -> Net-(D6-A)
- R24 pad 1: Net-(J11-CC1) -> +12V
- R24 pad 2: GND -> Net-(U11-FB)
- R25 pad 1: Net-(J12-CC1) -> Net-(U11-FB)
- R26 pad 1: Net-(D2-A) -> Net-(U11-RT/CLK)
- R26 pad 2: Net-(D1-A) -> GND
- R27 pad 1: Net-(D3-K) -> Net-(U11-COMP)
- R27 pad 2: Net-(U13-PA0) -> Net-(C37-Pad1)
- R28 pad 1: Net-(D4-K) -> Net-(D7-K)
- R28 pad 2: Net-(U13-PA1) -> Net-(D8-A)
- R29 pad 1: Net-(D5-K) -> Net-(D7-K)
- R29 pad 2: Net-(U13-PA4) -> Net-(U13-FB)
- R34 pad 1: +3.3V -> +24V
- R34 pad 2: Net-(D7-A) -> Net-(D10-A)
- R39 pad 1: +5V -> GND
- R39 pad 2: Net-(D9-A) -> Net-(Q5-G)
- R40 pad 1: +12V -> +24V
- R40 pad 2: Net-(D10-A) -> Net-(D12-A)
- R41 pad 1: /Connections/High Power Outputs 1/OUTA -> /Connections/High Power Outputs 2/OUTA
- R41 pad 2: Net-(Q1-G) -> Net-(Q6-G)
- R42 pad 1: /Connections/High Power Outputs 1/OUTB -> GND
- R42 pad 2: Net-(Q2-G) -> Net-(Q6-G)
- R43 pad 1: GND -> +24V
- R43 pad 2: Net-(Q1-G) -> Net-(D13-A)
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Routing:
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- added copper zone on B.Cu, net +24V
- added copper zone on F.Cu, net +24V
- added copper zone on In1.Cu, net +24V
- added copper zone on In2.Cu, net +24V
- added copper zone on In3.Cu, net +24V
- added copper zone on In4.Cu, net +24V
- added copper zone on B.Cu, net +3.3V
- added copper zone on F.Cu, net +3.3V
- added copper zone on B.Cu, net GND
- added copper zone on F.Cu, net GND
- added copper zone on In1.Cu, net GND
- added copper zone on In4.Cu, net GND
- added copper zone on B.Cu, net Net-(D10-A)
- added copper zone on F.Cu, net Net-(D10-A)
- added copper zone on In1.Cu, net Net-(D10-A)
- added copper zone on In2.Cu, net Net-(D10-A)
- added copper zone on In3.Cu, net Net-(D10-A)
- added copper zone on In4.Cu, net Net-(D10-A)
- added copper zone on F.Cu, net Net-(J28-Pin_1)
- added copper zone on F.Cu, net Net-(J28-Pin_2)
- added copper zone on F.Cu, net Net-(J28-Pin_3)
- added copper zone on F.Cu, net Net-(J28-Pin_4)
- added copper zone on F.Cu, net Net-(J29-Pin_1)
- added copper zone on F.Cu, net Net-(J29-Pin_2)
- added copper zone on F.Cu, net Net-(J29-Pin_3)
- added copper zone on F.Cu, net Net-(J29-Pin_4)
- added copper zone on F.Cu, net Net-(J30-Pin_1)
- added copper zone on F.Cu, net Net-(J30-Pin_2)
- added copper zone on F.Cu, net Net-(J30-Pin_3)
- added copper zone on F.Cu, net Net-(J31-Pin_1)
- added copper zone on F.Cu, net Net-(J31-Pin_2)
- added copper zone on F.Cu, net Net-(J31-Pin_3)
- added copper zone on F.Cu, net Net-(J32-Pin_2)
- added copper zone on F.Cu, net Net-(J33-Pin_1)
- added copper zone on F.Cu, net Net-(J33-Pin_2)
- added copper zone on F.Cu, net Net-(J33-Pin_3)
- added copper zone on F.Cu, net Net-(J33-Pin_4)
- added copper zone on F.Cu, net Net-(J38-Pin_2)
- added copper zone on F.Cu, net Net-(J39-Pin_2)
- added copper zone on F.Cu, net Net-(J40-Pin_2)
- added copper zone on F.Cu, net Net-(J46-Pin_1)
- added copper zone on F.Cu, net Net-(J46-Pin_3)
- added copper zone on F.Cu, net Net-(J46-Pin_4)
- added copper zone on F.Cu, net Net-(J47-Pin_1)
- added copper zone on F.Cu, net Net-(J47-Pin_3)
- added copper zone on F.Cu, net Net-(J47-Pin_4)
- added copper zone on F.Cu, net Net-(J48-Pin_1)
- added copper zone on F.Cu, net Net-(J48-Pin_3)
- added copper zone on F.Cu, net Net-(J48-Pin_4)
- added copper zone on F.Cu, net Net-(U24-CPI)
- added copper zone on F.Cu, net Net-(U24-CPO)
- added copper zone on F.Cu, net Net-(U24-IREF)
- added copper zone on F.Cu, net Net-(U24-VCP)
- added copper zone on F.Cu, net Net-(U24-VDD18)
- added copper zone on F.Cu, net Net-(U25-CPI)
- added copper zone on F.Cu, net Net-(U25-CPO)
- added copper zone on F.Cu, net Net-(U25-IREF)
- added copper zone on F.Cu, net Net-(U25-VCP)
- added copper zone on F.Cu, net Net-(U25-VDD18)
- added copper zone on F.Cu, net Net-(U26-CPI)
- added copper zone on F.Cu, net Net-(U26-CPO)
- added copper zone on F.Cu, net Net-(U26-IREF)
- added copper zone on F.Cu, net Net-(U26-VCP)
- added copper zone on F.Cu, net Net-(U26-VDD18)
- added copper zone on F.Cu, net Net-(U36-CPI)
- added copper zone on F.Cu, net Net-(U36-CPO)
- added copper zone on F.Cu, net Net-(U36-IREF)
- added copper zone on F.Cu, net Net-(U36-VCP)
- added copper zone on F.Cu, net Net-(U36-VDD18)
- added copper zone on F.Cu, net Net-(U43-CPI)
- added copper zone on F.Cu, net Net-(U43-CPO)
- added copper zone on F.Cu, net Net-(U43-IREF)
- added copper zone on F.Cu, net Net-(U43-VCP)
- added copper zone on F.Cu, net Net-(U43-VDD18)
- added copper zone on F.Cu, net Net-(U45-CPI)
- added copper zone on F.Cu, net Net-(U45-CPO)
- added copper zone on F.Cu, net Net-(U45-IREF)
- added copper zone on F.Cu, net Net-(U45-VCP)
- added copper zone on F.Cu, net Net-(U45-VDD18)
- added copper zone on F.Cu, net VM
Other:
- board outline added: 160 x 136 mm
- copper layers 4 -> 6
- board text added: "+"
- board text added: "-"
- board text added: "A"
- board text added: "B"
- board text added: "C"
- board text added: "DEBUG"
- board text added: "E1"
- board text added: "E2"
- board text added: "H1"
- board text added: "H2"
- board text added: "H3"
- board text added: "H4"
- board text added: "MOTOR"
- board text added: "USB"
- board text added: "X"
- board text added: "Y"
- board text added: "Z-PROBES"
- board text added: "Z1"
- board text added: "Z2"
- board text added: "Z3"
