File: lpo.kicad_sch (KiCad schematic)
At the start: 7 parts, among them J10 Conn_01x02, Q1 AO3400A

Commit message: ???
Parts:
- removed D14: LED_Small, APRLPrints:LED_0603, symbol Device:LED_Small
- removed D15: SS54, Diode_SMD:D_SMA, symbol Diode:SS38
- removed J10: Conn_01x02, Connector_Molex:Molex_Micro-Fit_3.0_43650-0215_1x02_P3.00mm_Vertical, symbol Connector_Generic:Conn_01x02
- removed Q1: AO3400A, Package_TO_SOT_SMD:SOT-23, symbol Transistor_FET:AO3400A
- removed R24: 10R, APRLPrints:R_0603, symbol Device:R_Small_US
- removed R25: 10k, APRLPrints:R_0603, symbol Device:R_Small_US
- removed R26: 100k, APRLPrints:R_0603, symbol Device:R_Small_US
- added D15: LED_Small, APRLPrints:LED_0603, symbol Device:LED_Small
- added J16: Conn_01x02, Connector_Molex:Molex_Micro-Fit_3.0_43650-0215_1x02_P3.00mm_Vertical, symbol Connector_Generic:Conn_01x02
- added Q5: AO3400A, Package_TO_SOT_SMD:SOT-23, symbol Transistor_FET:AO3400A
- added R41: 10R, APRLPrints:R_0603, symbol Device:R_Small_US
- added R42: 10k, APRLPrints:R_0603, symbol Device:R_Small_US
- added R43: 100k, APRLPrints:R_0603, symbol Device:R_Small_US
Connections:
- net +12V: now also J16.1 (Pin_1), R42.1
- net GND: now also Q5.2 (S), R43.1
- net OUT_LP: now also R41.1
- new net: D15.1 (K), J16.2 (Pin_2), Q5.3 (D)
- new net: D15.2 (A), R42.2
- new net: Q5.1 (G), R41.2, R43.2
Other:
- note added: "Low Power Output"

Commit message: loadcell math coming soon(tm)
Parts:
- J15: renamed from J16; footprint Connector_Molex:Molex_Micro-Fit_3.0_43650-0215_1x02_P3.00mm_Vertical -> Connector_JST:JST_XH_B2B-XH-AM_1x02_P2.50mm_Vertical
- renumbered R42 to R53, R41 to R54, R43 to R55
Changed lines of the file:
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@@
 		(dnp no)
 		(fields_autoplaced yes)
-		(property "Reference" "J16"
+		(property "Reference" "J15"
 			(at 142.24 96.5199 0)
 			(effects
@@
 			)
 		)
-		(property "Footprint" "Connector_Molex:Molex_Micro-Fit_3.0_43650-0215_1x02_P3.00mm_Vertical"
+		(property "Footprint" "Connector_JST:JST_XH_B2B-XH-AM_1x02_P2.50mm_Vertical"
 			(at 139.7 96.52 0)
 			(effects
@@
 			(project "Serie"
 				(path "/8fdbc9dc-a02a-488d-a5a6-6a3827681e3b/746d5c0a-0cd4-436a-8816-21d7d00bdf87/46d57e35-aa6e-4a67-a990-a23de73e2f99/2f1d21b0-0e1a-467e-9170-4eaa50b64fc6"
+					(reference "J16")
+					(unit 1)
+				)
+				(path "/8fdbc9dc-a02a-488d-a5a6-6a3827681e3b/746d5c0a-0cd4-436a-8816-21d7d00bdf87/46d57e35-aa6e-4a67-a990-a23de73e2f99/919e910d-a42d-4411-ad7a-daa09fd91ea9"
 					(reference "J17")
 					(unit 1)
 				)
-				(path "/8fdbc9dc-a02a-488d-a5a6-6a3827681e3b/746d5c0a-0cd4-436a-8816-21d7d00bdf87/46d57e35-aa6e-4a67-a990-a23de73e2f99/919e910d-a42d-4411-ad7a-daa09fd91ea9"
-					(reference "J18")
-					(unit 1)
-				)
 				(path "/8fdbc9dc-a02a-488d-a5a6-6a3827681e3b/746d5c0a-0cd4-436a-8816-21d7d00bdf87/46d57e35-aa6e-4a67-a990-a23de73e2f99/e6cfecc5-dd7f-413e-ae04-0f28b39e34b6"
-					(reference "J16")
+					(reference "J15")
 					(unit 1)
 				)
@@
 		(dnp no)
 		(fields_autoplaced yes)
-		(property "Reference" "R43"
+		(property "Reference" "R55"
 			(at 119.38 123.1899 0)
 			(effects
@@
 			(project "Serie"
 				(path "/8fdbc9dc-a02a-488d-a5a6-6a3827681e3b/746d5c0a-0cd4-436a-8816-21d7d00bdf87/46d57e35-aa6e-4a67-a990-a23de73e2f99/2f1d21b0-0e1a-467e-9170-4eaa50b64fc6"
-					(reference "R46")
+					(reference "R58")
 					(unit 1)
 				)
 				(path "/8fdbc9dc-a02a-488d-a5a6-6a3827681e3b/746d5c0a-0cd4-436a-8816-21d7d00bdf87/46d57e35-aa6e-4a67-a990-a23de73e2f99/919e910d-a42d-4411-ad7a-daa09fd91ea9"
-					(reference "R49")
+					(reference "R61")
 					(unit 1)
 				)
 				(path "/8fdbc9dc-a02a-488d-a5a6-6a3827681e3b/746d5c0a-0cd4-436a-8816-21d7d00bdf87/46d57e35-aa6e-4a67-a990-a23de73e2f99/e6cfecc5-dd7f-413e-ae04-0f28b39e34b6"
-					(reference "R43")
+					(reference "R55")
 					(unit 1)
 				)
@@
 		(dnp no)
 		(fields_autoplaced yes)
-		(property "Reference" "#PWR0133"
+		(property "Reference" "#PWR0132"
 			(at 130.81 99.06 0)
 			(effects
@@
 			(project "Serie"
 				(path "/8fdbc9dc-a02a-488d-a5a6-6a3827681e3b/746d5c0a-0cd4-436a-8816-21d7d00bdf87/46d57e35-aa6e-4a67-a990-a23de73e2f99/2f1d21b0-0e1a-467e-9170-4eaa50b64fc6"
-					(reference "#PWR0135")
+					(reference "#PWR0134")
 					(unit 1)
 				)
 				(path "/8fdbc9dc-a02a-488d-a5a6-6a3827681e3b/746d5c0a-0cd4-436a-8816-21d7d00bdf87/46d57e35-aa6e-4a67-a990-a23de73e2f99/919e910d-a42d-4411-ad7a-daa09fd91ea9"
-					(reference "#PWR0137")
+					(reference "#PWR0136")
 					(unit 1)
 				)
 				(path "/8fdbc9dc-a02a-488d-a5a6-6a3827681e3b/746d5c0a-0cd4-436a-8816-21d7d00bdf87/46d57e35-aa6e-4a67-a990-a23de73e2f99/e6cfecc5-dd7f-413e-ae04-0f28b39e34b6"
-					(reference "#PWR0133")
+					(reference "#PWR0132")
 					(unit 1)
 				)
@@
 		(dnp no)
 		(fields_autoplaced yes)
-		(property "Reference" "R42"
+		(property "Reference" "R53"
 			(at 119.38 99.0599 0)
 			(effects
@@
 			(project "Serie"
 				(path "/8fdbc9dc-a02a-488d-a5a6-6a3827681e3b/746d5c0a-0cd4-436a-8816-21d7d00bdf87/46d57e35-aa6e-4a67-a990-a23de73e2f99/2f1d21b0-0e1a-467e-9170-4eaa50b64fc6"
-					(reference "R45")
+					(reference "R56")
 					(unit 1)
 				)
 				(path "/8fdbc9dc-a02a-488d-a5a6-6a3827681e3b/746d5c0a-0cd4-436a-8816-21d7d00bdf87/46d57e35-aa6e-4a67-a990-a23de73e2f99/919e910d-a42d-4411-ad7a-daa09fd91ea9"
-					(reference "R48")
+					(reference "R59")
 					(unit 1)
 				)
 				(path "/8fdbc9dc-a02a-488d-a5a6-6a3827681e3b/746d5c0a-0cd4-436a-8816-21d7d00bdf87/46d57e35-aa6e-4a67-a990-a23de73e2f99/e6cfecc5-dd7f-413e-ae04-0f28b39e34b6"
-					(reference "R42")
+					(reference "R53")
 					(unit 1)
 				)
@@
 		(dnp no)
 		(fields_autoplaced yes)
-		(property "Reference" "#PWR0132"
+		(property "Reference" "#PWR0133"
 			(at 127 135.89 0)
 			(effects
@@
 			(project "Serie"
 				(path "/8fdbc9dc-a02a-488d-a5a6-6a3827681e3b/746d5c0a-0cd4-436a-8816-21d7d00bdf87/46d57e35-aa6e-4a67-a990-a23de73e2f99/2f1d21b0-0e1a-467e-9170-4eaa50b64fc6"
-					(reference "#PWR0134")
+					(reference "#PWR0135")
 					(unit 1)
 				)
 				(path "/8fdbc9dc-a02a-488d-a5a6-6a3827681e3b/746d5c0a-0cd4-436a-8816-21d7d00bdf87/46d57e35-aa6e-4a67-a990-a23de73e2f99/919e910d-a42d-4411-ad7a-daa09fd91ea9"
-					(reference "#PWR0136")
+					(reference "#PWR0137")
 					(unit 1)
 				)
 				(path "/8fdbc9dc-a02a-488d-a5a6-6a3827681e3b/746d5c0a-0cd4-436a-8816-21d7d00bdf87/46d57e35-aa6e-4a67-a990-a23de73e2f99/e6cfecc5-dd7f-413e-ae04-0f28b39e34b6"
-					(reference "#PWR0132")
+					(reference "#PWR0133")
 					(unit 1)
 				)
@@
 		(dnp no)
 		(fields_autoplaced yes)
-		(property "Reference" "R41"
+		(property "Reference" "R54"
 			(at 113.03 111.76 90)
 			(effects
@@
 			(project "Serie"
 				(path "/8fdbc9dc-a02a-488d-a5a6-6a3827681e3b/746d5c0a-0cd4-436a-8816-21d7d00bdf87/46d57e35-aa6e-4a67-a990-a23de73e2f99/2f1d21b0-0e1a-467e-9170-4eaa50b64fc6"
-					(reference "R44")
+					(reference "R57")
 					(unit 1)
 				)
 				(path "/8fdbc9dc-a02a-488d-a5a6-6a3827681e3b/746d5c0a-0cd4-436a-8816-21d7d00bdf87/46d57e35-aa6e-4a67-a990-a23de73e2f99/919e910d-a42d-4411-ad7a-daa09fd91ea9"
-					(reference "R47")
+					(reference "R60")
 					(unit 1)
 				)
 				(path "/8fdbc9dc-a02a-488d-a5a6-6a3827681e3b/746d5c0a-0cd4-436a-8816-21d7d00bdf87/46d57e35-aa6e-4a67-a990-a23de73e2f99/e6cfecc5-dd7f-413e-ae04-0f28b39e34b6"
-					(reference "R41")
-					(unit 1)
-				)
+					(reference "R54")
+					(unit 1)
+				)

Commit message: a
Parts:
- removed J15: Conn_01x02, Connector_JST:JST_XH_B2B-XH-AM_1x02_P2.50mm_Vertical, symbol Connector_Generic:Conn_01x02
- added D15: ESD9B3.3ST5G, Diode_SMD:D_SOD-923, symbol Diode:ESD9B3.3ST5G
- added J11: Conn_01x03, libserie:JST_XH_B3B-XH-AM_1x03_P2.50mm_Vertical, symbol Connector_Generic:Conn_01x03
- added R46: 10k, APRLPrints:R_0603, symbol Device:R_Small_US
- added R48: 4.7k, APRLPrints:R_0603, symbol Device:R_Small_US
- renumbered D15 to D14, Q5 to Q8, R53 to R47, R54 to R49, R55 to R50
Connections:
- net +12V: now also J11.1 (Pin_1)
- net GND: now also D15.1 (A1)
- net at D14.1 (K), Q8.3 (D): now also J11.2 (Pin_2)
- new net: J11.3 (Pin_3), R48.1
- new net +3.3V: R46.1
- new net TACH: D15.2 (A2), R46.2, R48.2
