File: sense.kicad_sch (KiCad schematic)
At the start: 58 parts, among them J10 Screw_Terminal_01x02, J3 Conn_01x02, J4 Conn_01x02, J5 Conn_01x02, J6 Conn_01x02, J7 Conn_01x04, J8 Conn_01x02, J9 Conn_01x02, U10 TLV6742, U4 LDC1612, U5 ADS1115IDGS, U6 ADS1220xPW, U7 TLV6742, U8 TMUX1101DBV, U9 TMUX1108PW

Commit message: loadcell math coming soon(tm)
Parts:
- removed J10: Screw_Terminal_01x02, Connector_Phoenix_MSTB:PhoenixContact_MSTBA_2,5_2-G_1x02_P5.00mm_Horizontal, symbol Connector_Generic:Conn_01x02
- added J6: Conn_01x02, Connector_PinHeader_1.00mm:PinHeader_1x02_P1.00mm_Vertical_SMD_Pin1Left, symbol Connector_Generic:Conn_01x02
- C10: footprint (none) -> APRLPrints:C_0603
- C11: renamed from C18; footprint (none) -> APRLPrints:C_0603
- C12: renamed from C14; footprint (none) -> APRLPrints:C_0603
- C13: renamed from C24; footprint (none) -> APRLPrints:C_0603
- C14: renamed from C27; footprint (none) -> APRLPrints:C_0603
- C15: renamed from C20; footprint (none) -> APRLPrints:C_0603
- C16: renamed from C7; footprint (none) -> APRLPrints:C_0603
- C17: renamed from C15; footprint (none) -> APRLPrints:C_0603
- C18: renamed from C26; footprint (none) -> APRLPrints:C_0603
- C19: renamed from C6; footprint (none) -> APRLPrints:C_0603
- C20: renamed from C8; footprint (none) -> APRLPrints:C_0603
- C21: renamed from C11; footprint (none) -> APRLPrints:C_0603
- C22: renamed from C16; footprint (none) -> APRLPrints:C_0603
- C23: renamed from C22; footprint (none) -> APRLPrints:C_0603
- C24: renamed from C9; footprint (none) -> APRLPrints:C_0603
- C25: renamed from C12; footprint (none) -> APRLPrints:C_0603
- C26: renamed from C17; footprint (none) -> APRLPrints:C_0603
- C27: renamed from C19; footprint (none) -> APRLPrints:C_0603
- C8: renamed from C25; footprint (none) -> APRLPrints:C_0603
- C9: renamed from C13; footprint (none) -> APRLPrints:C_0603
- J10: renamed from J6; footprint (none) -> Connector_PinHeader_1.00mm:PinHeader_1x02_P1.00mm_Vertical_SMD_Pin1Left
- J3: renamed from J7; footprint (none) -> Connector_PinHeader_1.00mm:PinHeader_1x04_P1.00mm_Vertical_SMD_Pin1Left
- J4: renamed from J8; footprint (none) -> Connector_PinHeader_1.00mm:PinHeader_1x02_P1.00mm_Vertical_SMD_Pin1Left
- J5: renamed from J9; footprint (none) -> Connector_PinHeader_1.00mm:PinHeader_1x02_P1.00mm_Vertical_SMD_Pin1Left
- J7: renamed from J3; footprint (none) -> Connector_PinHeader_1.00mm:PinHeader_1x02_P1.00mm_Vertical_SMD_Pin1Left
- J8: renamed from J4; footprint (none) -> Connector_PinHeader_1.00mm:PinHeader_1x02_P1.00mm_Vertical_SMD_Pin1Left
- J9: renamed from J5; footprint (none) -> Connector_PinHeader_1.00mm:PinHeader_1x02_P1.00mm_Vertical_SMD_Pin1Left
- R1: renamed from R3; footprint (none) -> APRLPrints:R_0603
- R10: renamed from R21; footprint (none) -> APRLPrints:R_0603
- R11, R2: footprint (none) -> APRLPrints:R_0603
- R12: renamed from R10; footprint (none) -> APRLPrints:R_0603
- R13: renamed from R12; footprint (none) -> APRLPrints:R_0603
- R14: renamed from R13; footprint (none) -> APRLPrints:R_0603
- R15: renamed from R1; footprint (none) -> APRLPrints:R_0603
- R16: renamed from R4; footprint (none) -> APRLPrints:R_0603
- R17: renamed from R5; footprint (none) -> APRLPrints:R_0603
- R18: renamed from R6; footprint (none) -> APRLPrints:R_0603
- R19: renamed from R7; footprint (none) -> APRLPrints:R_0603
- R20: renamed from R8; footprint (none) -> APRLPrints:R_0603
- R21: renamed from R9; footprint (none) -> APRLPrints:R_0603
- R3: renamed from R14; footprint (none) -> APRLPrints:R_0603
- R4: renamed from R15; footprint (none) -> APRLPrints:R_0603
- R5: renamed from R16; footprint (none) -> APRLPrints:R_0603
- R6: renamed from R17; footprint (none) -> APRLPrints:R_0603
- R7: renamed from R18; footprint (none) -> APRLPrints:R_0603
- R8: renamed from R19; footprint (none) -> APRLPrints:R_0603
- R9: renamed from R20; footprint (none) -> APRLPrints:R_0603
- U4: renamed from U7; footprint (none) -> Package_SO:SOIC-8_3.9x4.9mm_P1.27mm
- U5: renamed from U10; footprint (none) -> Package_SO:SOIC-8_3.9x4.9mm_P1.27mm
- renumbered C21 to C6, C23 to C7, U6 to U2, U9 to U3, U4 to U6, U8 to U7, U5 to U8
Connections:
- net GND: now also J6.1 (Pin_1)
- net at C18.1, R12.1, U4.2 (-)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: now also J6.2 (Pin_2)

Commit message: a
Parts:
- removed C24, C25, C26: 100nF, APRLPrints:C_0603, symbol Device:C_Small
- removed C27: 1uF, APRLPrints:C_0603, symbol Device:C_Small
- removed J10, J4, J5, J7, J8, J9: Conn_01x02, Connector_PinHeader_1.00mm:PinHeader_1x02_P1.00mm_Vertical_SMD_Pin1Left, symbol Connector_Generic:Conn_01x02
- removed R15, R16, R17, R18: 4.7k, APRLPrints:R_0603, symbol Device:R_Small_US
- removed R19, R20, R21: 10k, APRLPrints:R_0603, symbol Device:R_Small_US
- removed U8: ADS1115IDGS, Package_SO:TSSOP-10_3x3mm_P0.5mm, symbol Analog_ADC:ADS1115IDGS
- added C22: 100nF, APRLPrints:C_0603, symbol Device:C_Small
- added J5: Conn_01x04, libserie:JST_XH_B4B-XH-AM_1x04_P2.50mm_Vertical, symbol Connector_Generic:Conn_01x04
- added Y2: 12 MHz, APRLPrints:3225-4P-L, symbol Oscillator:IQXO-70
- C21: renamed from C22; value 1uF -> 100nF
- C23: value 100nF -> 30pF
- J4: renamed from J3; footprint Connector_PinHeader_1.00mm:PinHeader_1x04_P1.00mm_Vertical_SMD_Pin1Left -> libserie:JST_XH_B4B-XH-AM_1x04_P2.50mm_Vertical
- J6: footprint Connector_PinHeader_1.00mm:PinHeader_1x02_P1.00mm_Vertical_SMD_Pin1Left -> libserie:JST_XH_B2B-XH-AM_1x02_P2.50mm_Vertical
- U6: footprint Package_SON:WSON-12-1EP_4x4mm_P0.5mm_EP2.6x3mm_ThermalVias -> libserie:WSON-12-1EP_4x4mm_P0.5mm_EP2.6x3mm_ThermalVias
- renumbered C11 to C10, C12 to C11, C13 to C12, C14 to C13, C15 to C14, C16 to C15, C17 to C16, C18 to C17, C19 to C18, C20 to C19, C21 to C20, C6 to C5, C7 to C6, C8 to C7, C9 to C8, C10 to C9
Connections:
- net +3.3V: now also C22.1, Y2.4 (V+); no longer C23.1
- net GND: now also C22.2, Y2.2 (GND); no longer U6.3 (CLKIN)
- net at C16.2, C20.2, U6.11 (IN1A): now also J5.2 (Pin_2)
- net at C16.1, C21.2, U6.12 (IN1B): now also J5.1 (Pin_1)
- net at C15.1, C19.2, U6.10 (IN0B): now also J5.3 (Pin_3)
- net at C15.2, C18.2, U6.9 (IN0A): now also J5.4 (Pin_4)
- new net CLK: C23.1, U6.3 (CLKIN), Y2.3 (OUT)
- no-connect marks 2 -> 3
Other:
- note removed: "Extra Thermistor Inputs"
- note removed: "extra adc inputs"
