File: tc.kicad_sch (KiCad schematic)
At the start: 10 parts, among them J27 Conn_01x02, U13 MAX31856

Commit message: ???
Parts:
- removed C53, C55: 10n, APRLPrints:C_0603, symbol Device:C
- removed C54, C56, C57: 100n, APRLPrints:C_0603, symbol Device:C
- removed D16: LED, APRLPrints:LED_0603, symbol Device:LED
- removed R43, R44: 10k, APRLPrints:R_0603, symbol Device:R_US
- removed U13: MAX31856, Package_SO:TSSOP-14_4.4x5mm_P0.65mm, symbol MAX31856TriState:MAX31856
- added C72: 10nF, APRLPrints:C_0603, symbol Device:C
- added C73, C74: 100nF, APRLPrints:C_0603, symbol Device:C
- added D18: LED, APRLPrints:LED_0603, symbol Device:LED
- added R58: 4.02k, APRLPrints:R_0603, symbol Device:R_US
- added R59, R60: 10k, APRLPrints:R_0603, symbol Device:R_US
- added U22: MAX31865xTP, Package_DFN_QFN:TQFN-20-1EP_5x5mm_P0.65mm_EP3.25x3.25mm, symbol Sensor_Temperature:MAX31865xTP
Connections:
- net +3V3: now also C73.1, C74.1, R59.1, R60.1, U22.19 (DVDD), U22.20 (VDD)
- net GND: now also C73.2, C74.2, U22.10 (GND), U22.15 (DGND), U22.16 (GND), U22.21 (GND), U22.6 (FORCE2)
- net T1+: now also C72.1, U22.5 (FORCE+), U22.7 (RTDIN+)
- net T1-: now also C72.2, U22.8 (RTDIN-), U22.9 (FORCE-)
- net TC_MISO: now also U22.14 (SDO)
- net TC_MOSI: now also U22.11 (SDI)
- net TC_SCK: now also U22.12 (SCLK)
- net ~{CS}: now also R59.2, U22.13 (~{CS})
- net ~{DRDY}: now also D18.1 (K), U22.18 (~{DRDY})
- new net: D18.2 (A), R60.2
- new net: R58.1, U22.1 (BIAS), U22.2 (REFIN+)
- new net: R58.2, U22.3 (REFIN-), U22.4 (ISENSOR)
Other:
- note added: "Should be 0.1%"
- note added: "Thermocouple"
- note added: "should be jst xh, 2 pin"

Commit message: loadcell math coming soon(tm)
Parts:
- J26: renamed from J27; footprint Connector_Molex:Molex_Micro-Fit_3.0_43650-0215_1x02_P3.00mm_Vertical -> Connector_JST:JST_XH_B2B-XH-AM_1x02_P2.50mm_Vertical
- renumbered C73 to C72, C74 to C73, C72 to C74, R60 to R70, R59 to R71, R58 to R72, U22 to U20

Commit message: a
Parts:
- J22: renamed from J26; footprint Connector_JST:JST_XH_B2B-XH-AM_1x02_P2.50mm_Vertical -> libserie:JST_XH_B2B-XH-AM_1x02_P2.50mm_Vertical
- U22: renamed from U20; footprint Package_DFN_QFN:TQFN-20-1EP_5x5mm_P0.65mm_EP3.25x3.25mm -> libserie:TQFN-20-1EP_5x5mm_P0.65mm_EP3.25x3.25mm
- renumbered C72 to C76, C73 to C77, C74 to C78, D18 to D20, R70 to R69, R71 to R70, R72 to R71
Connections:
- net +3V3 renamed +3.3V
- net ~{DRDY}: no longer names the net of D20.1 (K), U22.18 (~{DRDY})
Other:
- note added: "Microcontroller does not use ~{DRDY}"
